File: projects/usb-power-3s/04_kicad/usb_power_3s.kicad_pcb (KiCad board)
At the start: 4 copper layers, 100 x 60 mm, 100 parts, among them J1 XT60_BATT, J2 USB-A 2.5A, J3 USB-A 2.5A, J4 USB-A 2.5A, J5 USB4105-GF-A, Q1 CSD18543Q3A diode, Q2 CSD18543Q3A switch, U1 LM74800-Q1, U2 LM5145 rail A, U3 LM5145 rail B, U4 TPS2557 2.5A, U5 TPS2557 2.5A, U6 TPS2557 2.5A

Commit message: usb-power-3s v1.1: LM5145 footprint was MIRROR-NUMBERED - fixed + re-routed
The new jlc_twin stage (D5) compares our footprints against JLCPCB's own CAD
(easyeda2kicad) on its first run found the vendored VQFN-20 winding CW vs the
datasheet's CCW - a dead-board defect invisible to every electrical check.
Pads renumbered n->21-n, chain re-routed with taps hardest-first (KRT temp-net
waves TAPB/C/F/G/H/U/V/W), robust tail-trimmer/via-janitor/hair-gap-snap
passes, gate green: DRC 0 violations / 0 unconnected / 0 parity.

WARNING: SPF power_board_v1 (ordered 2026-07-14) shares this footprint on
U1/U2 - those boards' buck controllers will not function.

Co-Authored-By: Claude Opus 4.8 <noreply@anthropic.com>
Routing:
- net 5V_A: track 55.4 -> 180.8 mm, vias 24 -> 22
- net VSW: track 1.60 -> 73.5 mm
- net EN_A: track 18.7 -> 47.9 mm, vias 4 -> 5
- net FE_MID: track 25.3 -> 53.9 mm, vias 13 -> 19
- net VBATT_F: track 0.00 -> 24.8 mm, vias 10 -> 14
- net 5V_C: track 81.2 -> 104.3 mm, vias 19 -> 16
- net FB_A: track 32.7 -> 51.4 mm, vias 6 -> 4
- net PGOOD_A: track 45.2 -> 59.8 mm
- net BST_B: track 40.1 -> 26.3 mm, vias 2 -> 4
- net FB_B: track 40.4 -> 51.2 mm, vias 6 -> 4
- net SS_A: track 42.5 -> 31.8 mm, vias 4 -> 0
- net COMP_A: track 31.5 -> 41.1 mm, vias 3 -> 4
- net SW_A: track 46.1 -> 37.0 mm, vias 11 -> 10
- net BST_A: track 40.4 -> 31.6 mm, vias 0 -> 2
- net LO_A: track 8.96 -> 17.6 mm
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- added copper zone on B.Cu, net 5V_C
