File: projects/usb-power-3s/04_kicad/usb_power_3s.kicad_sch (KiCad schematic)
At the start: 96 parts, among them J1 XT60_BATT, J2 USB-A 2.5A, J3 USB-A 2.5A, J4 USB-A 2.5A, J5 USB4105-GF-A, Q1 CSD18543Q3A diode, Q2 CSD18543Q3A switch, U1 LM74800-Q1, U2 LM5145 rail A, U3 LM5145 rail B, U4 TPS2557 2.5A, U5 TPS2557 2.5A, U6 TPS2557 2.5A

Commit message: usb-power-3s: retrofit policy gates — 6 FAILs -> 0 (4 evidence-backed waivers)
Released board (v1.1-2026-07-16): fab outputs untouched (04_kicad board
copper/silk unchanged; netlist parity 0, DRC 0/0/0 at severity-all).

- S-VER: 4 weak part.yaml notes rewritten from the actual pinout figures.
  CSD18543Q3A (cached SLPS432.pdf is really SLPS633 p.1 Top View, noted),
  TPS2557 (SLVS931B sec.6 p.3), USB4105-GF-A + 1001-011-01101 drawings
  fetched, sha256-pinned and committed (CNC drawing is mechanical-only —
  note says so honestly). New gotcha: GCT drawing rates VBUS 5.00A
  collectively vs the board's 6A-copper claim.
- P-POL: audit_board.py I9 asserts pad-1 nets of all 10 polarized parts
  (XT60, 3x TVS, 2x LED, 3x CP_Elec) against part.yaml facts; passes.
- S-ERC/S-NC: generate_schematic.py emits 13 no_connect flags for the
  sanctioned floats (U2/U3 SYNCOUT+NC, U4-U6 FAULT, J5 SBU — each
  re-verified vs pin_review.md + datasheets). ERC errors 13 -> 0.
  Warnings 193 -> 97: pwr.kicad_sym + sym-lib-table clears the 96
  lib_symbol_issues; remainder baselined with reasons
  (rules/erc_warning_baseline.yaml). rebuild_all.sh gains the ERC gate.
- R-RULES: new 03_src/route_prep.py builds future route-input projects
  carrying the netclasses+floors (refuses tracked/filled boards);
  historical r0 left as-shipped, adopted-forward waiver.
- R-POUR: VBUS1-3 measured 0.8mm/1oz continuous F.Cu (vias only feed the
  port-cap spur). At 2.51A ILIM worst case: ~16C rise, but 1.5x margin
  NOT met (1.32x @30C) — recorded honestly as a next-spin defect.
- P-SILK-REF/P-SILK-FN: adopted-forward waivers (policies postdate the
  release); next-spin remediation listed.

policy_audit FULL: was FAIL=6 -> now FAIL=0 (PASS=13, WAIVED=4, HUMAN=6,
N-A=2), incl. S-ERC/S-NC/P-CRT/R-DRC now graded PASS with DRC enabled.

Co-Authored-By: Claude Fable 5 <noreply@anthropic.com>
Connections:
- no-connect marks 0 -> 13
