File: projects/crowsync-recorder/04_kicad/crowsync_recorder.kicad_sch (KiCad schematic)
At the start: 51 parts, among them J1 USB4105-GF-A, J2 JST-GH mic, J3 JST-GH PPS, U1 PCM2900CDBR, U2 TLV9062IDR, U3 TPS7A2033PDBVR, Y1 12MHz 3225 20pF

Commit message: crowsync-recorder: retrofit policy gates — P-POL, S-ERC, S-NC now enforced
- audit_board.py I9: scripted pad-1-net polarity check (D3/D4 LEDs pad1=K=GND,
  D1/D2 USBLC6 GND/rail refs + pass-through pair coherence) from part.yaml facts
- generate_schematic.py: emit no_connect flags for the 9 sanctioned floats
  (J1 SBU1/2, U3 NC, U1 HID0-2/TEST1/VOUTL/VOUTR — each verified against
  v1.0 pin_review.md + ORDER_README oddities); asserts emitted NC set ==
  sanctioned list so new accidental floats fail the build
- generate project csr.kicad_sym + sym-lib-table: kills 51 lib_symbol_issues
- rebuild_all.sh: ERC gate at --severity-all, 0 errors; warnings baselined
  to endpoint_off_grid only (reason in script)
- ERC: 9 errors/102 warnings -> 0 errors/51 baselined warnings
- netlist parity node-for-node identical (44 nets); board DRC+parity 0/0/0;
  04_kicad board untouched. policy_audit: FAIL 3 -> 0

Co-Authored-By: Claude Fable 5 <noreply@anthropic.com>
Connections:
- no-connect marks 0 -> 9
