File: projects/shitty-kitty/06_build/route/w1.kicad_pcb (KiCad board)
At the start: 4 copper layers, 130 x 75 mm, 82 parts, among them J1 DC-005C-20A 12V, J2 TYPE-C-31-M-12, J3 ELECTRODES INNER, J4 ELECTRODES OUTER, J5 MOTOR NEMA17, J6 ENDSTOP TERM, J8 HOST 1x6, Q1 AOD4185 revpol, SW1 TS-1187A BOOT, SW2 TS-1187A RESET, U1 ESP32-S3-WROOM-1-N8R2, U2 TMC2209-LA-T, U3 MPR121QR2 0x5A, U4 MPR121QR2 0x5B, U5 MPR121QR2 0x5C, U6 MPR121QR2 0x5D, U7 LIS2DH12TR, U8 AP63205WU-7, U9 AMS1117-3.3

Commit message: shitty-kitty: route iteration — MPR121s rotated 90 (electrodes north/east, support south), single mega signal wave (intra-wave ripup arbitration), BRA/BRB ride the motor wave
Co-Authored-By: Claude Fable 5 <noreply@anthropic.com>
Routing:
- net VIN_F: track 0.00 -> 19.8 mm
- net VIN_RAW: track 0.00 -> 9.75 mm
Changed lines of the file:
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@@
 	)
 	(embedded_fonts no)
+	(segment
+		(start 166.500000 70.000000)
+		(end 160.350000 63.850000)
+		(width 0.8)
+		(layer "F.Cu")
+		(net "VIN_RAW")
+	)
+	(segment
+		(start 160.350000 63.850000)
+		(end 160.350000 62.800000)
+		(width 0.8)
+		(layer "F.Cu")
+		(net "VIN_RAW")
+	)
+	(segment
+		(start 164.650000 62.800000)
+		(end 164.650000 62.950000)
+		(width 0.8)
+		(layer "F.Cu")
+		(net "VIN_F")
+	)
+	(segment
+		(start 164.650000 62.950000)
+		(end 168.450000 66.750000)
+		(width 0.8)
+		(layer "F.Cu")
+		(net "VIN_F")
+	)
+	(segment
+		(start 168.450000 66.750000)
+		(end 168.450000 70.200000)
+		(width 0.8)
+		(layer "F.Cu")
+		(net "VIN_F")
+	)
+	(segment
+		(start 168.450000 70.200000)
+		(end 168.350000 70.300000)
+		(width 0.8)
+		(layer "F.Cu")
+		(net "VIN_F")
+	)
+	(segment
+		(start 168.350000 70.300000)
+		(end 168.350000 70.550000)
+		(width 0.8)
+		(layer "F.Cu")
+		(net "VIN_F")
+	)
+	(segment
+		(start 168.350000 70.550000)
+		(end 168.250000 70.650000)
+		(width 0.8)
+		(layer "F.Cu")
+		(net "VIN_F")
+	)
+	(segment
+		(start 168.250000 70.650000)
+		(end 168.250000 70.700000)
+		(width 0.8)
+		(layer "F.Cu")
+		(net "VIN_F")
+	)
+	(segment
+		(start 168.250000 70.700000)
+		(end 168.150000 70.800000)
+		(width 0.8)
+		(layer "F.Cu")
+		(net "VIN_F")
+	)
+	(segment
+		(start 168.150000 70.800000)
+		(end 168.150000 70.850000)
+		(width 0.8)
+		(layer "F.Cu")
+		(net "VIN_F")
+	)
+	(segment
+		(start 168.150000 70.850000)
+		(end 168.050000 70.950000)
+		(width 0.8)
+		(layer "F.Cu")
+		(net "VIN_F")
+	)
+	(segment
+		(start 168.050000 70.950000)
+		(end 168.050000 71.000000)
+		(width 0.8)
+		(layer "F.Cu")
+		(net "VIN_F")
+	)
+	(segment
+		(start 168.050000 71.000000)
+		(end 163.800000 75.250000)
+		(width 0.8)
+		(layer "F.Cu")
+		(net "VIN_F")
+	)
+	(segment
+		(start 163.800000 75.250000)
+		(end 160.000000 75.250000)
+		(width 0.8)
+		(layer "F.Cu")
+		(net "VIN_F")
+	)
 )
