File: projects/shitty-kitty/06_build/route/w1b.kicad_pcb (KiCad board)
At the start: 4 copper layers, 130 x 75 mm, 82 parts, among them J1 DC-005C-20A 12V, J2 TYPE-C-31-M-12, J3 ELECTRODES INNER, J4 ELECTRODES OUTER, J5 MOTOR NEMA17, J6 ENDSTOP TERM, J8 HOST 1x6, Q1 AOD4185 revpol, SW1 TS-1187A BOOT, SW2 TS-1187A RESET, U1 ESP32-S3-WROOM-1-N8R2, U2 TMC2209-LA-T, U3 MPR121QR2 0x5A, U4 MPR121QR2 0x5B, U5 MPR121QR2 0x5C, U6 MPR121QR2 0x5D, U7 LIS2DH12TR, U8 AP63205WU-7, U9 AMS1117-3.3

Commit message: shitty-kitty: WIP CHECKPOINT (not a gate) — routing surgery mid-flight, 18 DRC violations remain (6 clearance/5 hole_clr/6 h2h/1 conn_width from the SDA-via relocation), 0 unconnected. Route-surgery tooling: route_taps/route_unlock/lift_floors. Agent died on Fable credit wall; preserving work
Co-Authored-By: Claude Fable 5 <noreply@anthropic.com>
Routing:
- net V5OUT: track 0.00 -> 7.17 mm
- net VCP: track 0.00 -> 5.16 mm
- net CPO: track 0.00 -> 5.12 mm
- net CPI: track 0.00 -> 3.43 mm, vias 0 -> 2
Changed lines of the file:
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@@
 		(net "VIN_F")
 	)
+	(segment
+		(start 157.550000 104.000000)
+		(end 155.950000 104.000000)
+		(width 0.25)
+		(layer "F.Cu")
+		(net "VCP")
+	)
+	(segment
+		(start 155.950000 104.000000)
+		(end 155.450000 103.500000)
+		(width 0.25)
+		(layer "F.Cu")
+		(net "VCP")
+	)
+	(segment
+		(start 155.450000 103.500000)
+		(end 155.300000 103.500000)
+		(width 0.25)
+		(layer "F.Cu")
+		(net "VCP")
+	)
+	(segment
+		(start 155.300000 103.500000)
+		(end 155.250000 103.450000)
+		(width 0.25)
+		(layer "F.Cu")
+		(net "VCP")
+	)
+	(segment
+		(start 155.250000 103.450000)
+		(end 154.100000 103.450000)
+		(width 0.25)
+		(layer "F.Cu")
+		(net "VCP")
+	)
+	(segment
+		(start 154.100000 103.450000)
+		(end 153.050000 104.500000)
+		(width 0.25)
+		(layer "F.Cu")
+		(net "VCP")
+	)
+	(segment
+		(start 157.550000 103.000000)
+		(end 154.550000 103.000000)
+		(width 0.25)
+		(layer "F.Cu")
+		(net "CPO")
+	)
+	(segment
+		(start 154.550000 103.000000)
+		(end 153.050000 101.500000)
+		(width 0.25)
+		(layer "F.Cu")
+		(net "CPO")
+	)
+	(segment
+		(start 157.550000 103.500000)
+		(end 156.450000 102.400000)
+		(width 0.25)
+		(layer "B.Cu")
+		(net "CPI")
+	)
+	(segment
+		(start 156.450000 102.400000)
+		(end 155.550000 101.500000)
+		(width 0.25)
+		(layer "F.Cu")
+		(net "CPI")
+	)
+	(segment
+		(start 155.550000 101.500000)
+		(end 154.950000 101.500000)
+		(width 0.25)
+		(layer "F.Cu")
+		(net "CPI")
+	)
+	(via
+		(at 156.450000 102.400000)
+		(size 0.6)
+		(drill 0.3)
+		(layers "F.Cu" "B.Cu")
+		(tenting (front yes) (back yes))
+		(net "CPI")
+	)
+	(via
+		(at 157.537500 103.500000)
+		(size 0.45)
+		(drill 0.3)
+		(layers "F.Cu" "B.Cu")
+		(tenting (front yes) (back yes))
+		(net "CPI")
+	)
+	(segment
+		(start 158.500000 105.450000)
+		(end 155.450000 108.500000)
+		(width 0.25)
+		(layer "F.Cu")
+		(net "V5OUT")
+	)
+	(segment
+		(start 155.450000 108.500000)
+		(end 155.300000 108.500000)
+		(width 0.25)
+		(layer "F.Cu")
+		(net "V5OUT")
+	)
+	(segment
+		(start 155.300000 108.500000)
+		(end 155.250000 108.550000)
+		(width 0.25)
+		(layer "F.Cu")
+		(net "V5OUT")
+	)
+	(segment
+		(start 155.250000 108.550000)
+		(end 154.100000 108.550000)
+		(width 0.25)
+		(layer "F.Cu")
+		(net "V5OUT")
+	)
+	(segment
+		(start 154.100000 108.550000)
+		(end 153.050000 107.500000)
+		(width 0.25)
+		(layer "F.Cu")
+		(net "V5OUT")
+	)
 )
