File: projects/shitty-kitty/06_build/route/w2b1.kicad_pcb (KiCad board)
At the start: 4 copper layers, 130 x 75 mm, 82 parts, among them J1 DC-005C-20A 12V, J2 TYPE-C-31-M-12, J3 ELECTRODES INNER, J4 ELECTRODES OUTER, J5 MOTOR NEMA17, J6 ENDSTOP TERM, J8 HOST 1x6, Q1 AOD4185 revpol, SW1 TS-1187A BOOT, SW2 TS-1187A RESET, U1 ESP32-S3-WROOM-1-N8R2, U2 TMC2209-LA-T, U3 MPR121QR2 0x5A, U4 MPR121QR2 0x5B, U5 MPR121QR2 0x5C, U6 MPR121QR2 0x5D, U7 LIS2DH12TR, U8 AP63205WU-7, U9 AMS1117-3.3

Commit message: shitty-kitty: WIP CHECKPOINT (not a gate) — routing surgery mid-flight, 18 DRC violations remain (6 clearance/5 hole_clr/6 h2h/1 conn_width from the SDA-via relocation), 0 unconnected. Route-surgery tooling: route_taps/route_unlock/lift_floors. Agent died on Fable credit wall; preserving work
Co-Authored-By: Claude Fable 5 <noreply@anthropic.com>
Routing:
- net 3V3: track 305.3 -> 0.00 mm, vias 18 -> 0
- net SCL: track 127.5 -> 0.00 mm, vias 24 -> 0
- net SDA: track 107.4 -> 0.00 mm, vias 14 -> 0
- net 5V: track 83.8 -> 0.00 mm, vias 5 -> 0
- net USB_DP: track 75.7 -> 0.00 mm, vias 6 -> 0
- net ENN: track 74.1 -> 0.00 mm, vias 4 -> 0
- net ENDSTOP_G: track 73.0 -> 0.00 mm, vias 2 -> 0
- net DIR: track 72.8 -> 0.00 mm, vias 2 -> 0
- net STEP: track 72.0 -> 0.00 mm
- net USB_DM: track 71.5 -> 0.00 mm, vias 6 -> 0
- net MPR_IRQ1: track 67.5 -> 0.00 mm, vias 6 -> 0
- net EN: track 67.3 -> 0.00 mm, vias 8 -> 0
- net DIAG: track 65.4 -> 0.00 mm
- net TMC_UART: track 62.6 -> 0.00 mm, vias 4 -> 0
- net INDEX: track 60.4 -> 0.00 mm, vias 2 -> 0
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