File: projects/crow-array-central/06_build/route/r2.kicad_pcb (KiCad board)
At the start: 6 copper layers, 176 x 122 mm, 238 parts, among them J1 RJHSE-5384, J10 INJ IN, J11 5V TERM DNP, J12 USB4105-GF-A, J13 xSYS DBG TDI/TDO, J14 xSYS DBG TMS/TCK, J2 RJHSE-5384, J3 RJHSE-5384, J4 RJHSE-5384, J5 RJHSE-5384, J6 RJHSE-5384, J7 RJHSE-5384 DNP, J8 RJHSE-5384 DNP, J9 DC-005 5V IN, Q1 AO3400A beep 1, Q2 AO3400A beep 2, Q3 AO3400A beep 3, Q4 AO3400A beep 4, Q5 AO3400A beep 5, Q6 AO3400A beep 6, Q7 AO3400A beep 7, Q8 AO3400A beep 8, Q9 AO3401A revFET, U1 XU316-1024-TQ128-I24, U10 AP61102 3V3, U11 AP61102 0V9, U12 TCR2LF18 1V8, U13 XC6227 3V3A, U2 PCM1865DBTR, U3 PCM1865DBTR, U4 W25Q16JVSSIQ, U5 NC7NZ34 MCLK buf, U6 SHT40-AD1B (0x44), Y1 FA-238 24MHz

Commit message: crow-array-central: DRC cleanup 101->32+5 (parity 0); Q9 polarity confirmed; small-via tier ADR-0009
DRU set to JLC 6L real capability (D20): clearance/track 0.09, hole-to-hole 0.2
edge, via 0.30/0.15 (small-via option, ADR-0009). Fixed ALL shorts (TDO/TDI
escape dogbone), hole_to_hole, hole_clearance, lib_footprint_mismatch (SHT40
vendored), silk_edge (J9 barrel silk clamped). GND pad rescue 15->5 unconnected.
Q9 AO3401A polarity CONFIRMED correct on board by dedicated datasheet review;
fixed two wrong part.yaml notes to agree with datasheet+ADR-0007. Residual:
18 clearance (sub-0.09 power-vs-signal) + 14 dangling (loose copper) + 5
unconnected GND = KRT route-quality rework, NOT 0/0/0 yet (documented in BRIEF).

Co-Authored-By: Claude Fable 5 <noreply@anthropic.com>
Parts:
- J9: footprint cac:BarrelJack_Horizontal -> Connector_BarrelJack:BarrelJack_Horizontal
- U6: footprint cac:Sensirion_DFN-4_1.5x1.5mm_P0.8mm_SHT4x_NoCentralPad -> Sensor_Humidity:Sensirion_DFN-4_1.5x1.5mm_P0.8mm_SHT4x_NoCentralPad
Routing:
- net I2C_SCL: track 215.4 -> 7.54 mm, vias 7 -> 0
- net I2C_SDA: track 144.7 -> 7.48 mm, vias 7 -> 0
- net AIN_P4: track 106.3 -> 0.00 mm, vias 3 -> 0
- net LRCK: track 99.7 -> 2.68 mm, vias 3 -> 0
- net BCLK: track 99.3 -> 4.43 mm, vias 6 -> 0
- net BEEP_G1: track 95.8 -> 3.72 mm, vias 2 -> 0
- net 3V3: track 475.7 -> 389.4 mm, vias 21 -> 12
- net TMS: track 86.5 -> 2.16 mm, vias 1 -> 0
- net AUD_P1: track 82.3 -> 0.00 mm, vias 2 -> 0
- net TCK: track 82.6 -> 1.85 mm, vias 2 -> 0
- net BEEP_G8: track 81.9 -> 2.07 mm, vias 2 -> 0
- net TDO: track 80.5 -> 4.06 mm, vias 1 -> 0
- net BEEP_G2: track 78.4 -> 2.90 mm, vias 4 -> 0
- net TDI: track 77.4 -> 4.40 mm, vias 1 -> 0
- net BEEP_G3: track 73.9 -> 2.16 mm, vias 2 -> 0
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