File: projects/crow-array-pod/06_build/route/r3.kicad_pcb (KiCad board)
At the start: 2 copper layers, 94.5 x 44.5 mm, 40 parts, among them J1 RJHSE-5384, J2 MIC PADS (AOM-5024L), U1 OPA1678IDR

Commit message: WIP CHECKPOINT (not a gate) — pod v1.1 verification-phase files + cook-hub project skeleton; agents interrupted, preserving state before relaunch
Co-Authored-By: Claude Fable 5 <noreply@anthropic.com>
Parts:
- moved L1 18.7 mm to (93.7, 54.2)
- moved D1 9.70 mm to (88.5, 68.7)
- moved J1 7.00 mm to (78.0, 71.0), turned to 90 degrees
Routing:
- net 5V: track 120.0 -> 85.4 mm, vias 7 -> 3
- net SHIELD: track 45.7 -> 34.8 mm, vias 3 -> 0
- net AUDIO_N: track 51.3 -> 61.6 mm, vias 4 -> 5
- net AUDIO_P: track 49.8 -> 58.4 mm, vias 0 -> 7
- net AUD_N_I: track 13.2 -> 21.7 mm, vias 2 -> 4
- net FB_B: track 20.8 -> 29.0 mm
- net BEEP_RET: track 46.9 -> 39.0 mm, vias 0 -> 1
- net BEEP_5V: track 26.7 -> 20.0 mm, vias 2 -> 0
- net MIC: track 46.9 -> 41.4 mm, vias 0 -> 2
- net B_OUT: track 27.4 -> 31.9 mm
- net AUD_P_I: track 19.3 -> 15.3 mm
- net AIN: track 13.4 -> 11.4 mm, vias 3 -> 4
- net 5VF: track 56.9 -> 55.5 mm, vias 2 -> 0
- net FB_A: track 17.8 -> 18.6 mm
- net A_OUT: track 23.2 -> 22.5 mm, vias 2 -> 0
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