File: projects/cook-hub/04_kicad/cook_hub.kicad_sch (KiCad schematic)
At the start: 176 parts, among them J1 EXT 5V 2A, J10 CONTACTOR 30V, J11 X9555WV 2x16 KEYPAD, J12 ENCODER DNP, J13 STEP/DIR/EN DNP, J14 SPARE I2C0+GP4, J15 MAX31865 DNP, J2 Pico 2 socket, J3 I2C0 MLX+SHT45, J4 I2C1 EXHAUST SHT45, J5 TC K-TYPE, J6 LOADCELL DIG, J7 DOOR NC+EOL, J8 E-STOP NC, J9 NTC x3, K1 DIP05-1A72-12L, K10 DIP05-1A72-12L, K11 DIP05-1A72-12L, K12 DIP05-1A72-12L, K13 DIP05-1A72-12L, K14 DIP05-1A72-12L, K15 DIP05-1A72-12L, K16 DIP05-1A72-12L, K2 DIP05-1A72-12L, K3 DIP05-1A72-12L, K4 DIP05-1A72-12L, K5 DIP05-1A72-12L, K6 DIP05-1A72-12L, K7 DIP05-1A72-12L, K8 DIP05-1A72-12L, K9 DIP05-1A72-12L, Q1 AO3401A hi-side, Q2 2N7002, Q3 AO3401A rev-prot, SW1 RUN reset, U1 MAX31856, U10 LTV-817S, U11 74HC14 E-stop, U12 AMS1117-3.3, U13 USBLC6-2SC6, U14 USBLC6-2SC6, U15 USBLC6-2SC6, U3 74HC595 #1, U4 74HC595 #2, U5 ULN2803A K1-K8, U6 ULN2803A K9-K16, U7 SN74LVC1G123, U8 74LVC1G00 /OE, U9 74LVC1G11 AND3

Commit message: cook-hub: WIP CHECKPOINT (not a gate) — board placement/route iteration in flight (U5 west move pending); agent hit session limit
Co-Authored-By: Claude Fable 5 <noreply@anthropic.com>
Parts:
- TP41, TP42, TP43, TP44, TP45, TP46, TP47, TP48, TP49, TP50, TP51, TP52, TP53, TP54, TP55, TP56: footprint TestPoint:TestPoint_THTPad_D2.0mm_Drill1.0mm -> TestPoint:TestPoint_Pad_D1.5mm

Commit message: cook-hub: GATE GREEN again after D-FIX U7 (twin-caught wrong-pitch footprint)
The jlc_twin PAD-GEOM check caught a DEAD-BOARD defect the whole gate stack
missed: U7 SN74LVC1G123DCTR is a DCT SSOP-8 at 0.65mm pitch, but the board
carried Package_SO:SSOP-8_3.9x5.05mm_P1.27mm (1.27mm pitch) — self-
consistent in netlist/DRC/parity, unassemblable in reality (ours 6.57mm
across vs JLC's 4.10mm). Fix: Package_SO:SSOP-8_2.95x2.8mm_P0.65mm (pad1-5
3.92mm, matches the DS land). The sealed schematic's net topology is
untouched — only the footprint field changed (documented D-FIX).

Repair strategy (fresh 0.21 reroute scored worse — 2 shorts): champion
patchwork chain restored from git; U7's footprint block SPLICED into the
chain textually; WD nets stripped + KRT-repaired (WD_OK/CX/RCX at 0.21,
WD_PULSE at 0.13/0.2); stale 3V3 pocket feeds stripped; sub-floor track
widener; A*-via annulus bump (pcb_toolkit's 0.45/0.2 default = 0.125
annular < the 0.13 floor); post_sweep near-dup via dedupe; fixups.py — a
deterministic named-site rescue pass (U7.3 + R21.2 pour-bond via+stub,
exact-collide green at runtime, hard-fail if a site goes stale) + frayed-
trunk re-termination onto C15.1; named DRU exemption area u7_taps with a
scoped 0.25mm PWR floor (crow neck_approaches pattern, <15mA taps).

Gate: DRC severity-all --refill-zones --schematic-parity 0/0/0, rebuild
exit 0, ERC 0, AUDIT PASS. Chain promoted (canon M3).

Co-Authored-By: Claude Fable 5 <noreply@anthropic.com>
Parts:
- U7: footprint Package_SO:SSOP-8_3.9x5.05mm_P1.27mm -> Package_SO:SSOP-8_2.95x2.8mm_P0.65mm
