File: projects/cook-hub/06_build/route/r1.kicad_pcb (KiCad board)
At the start: 4 copper layers, 185 x 112 mm, 182 parts, among them J1 EXT 5V 2A, J10 CONTACTOR 30V, J11 X9555WV 2x16 KEYPAD, J12 ENCODER DNP, J13 STEP/DIR/EN DNP, J14 SPARE I2C0+GP4, J15 MAX31865 DNP, J2 Pico 2 socket, J3 I2C0 MLX+SHT45, J4 I2C1 EXHAUST SHT45, J5 TC K-TYPE, J6 LOADCELL DIG, J7 DOOR NC+EOL, J8 E-STOP NC, J9 NTC x3, K1 DIP05-1A72-12L, K10 DIP05-1A72-12L, K11 DIP05-1A72-12L, K12 DIP05-1A72-12L, K13 DIP05-1A72-12L, K14 DIP05-1A72-12L, K15 DIP05-1A72-12L, K16 DIP05-1A72-12L, K2 DIP05-1A72-12L, K3 DIP05-1A72-12L, K4 DIP05-1A72-12L, K5 DIP05-1A72-12L, K6 DIP05-1A72-12L, K7 DIP05-1A72-12L, K8 DIP05-1A72-12L, K9 DIP05-1A72-12L, Q1 AO3401A hi-side, Q2 2N7002, Q3 AO3401A rev-prot, SW1 RUN reset, U1 MAX31856, U10 LTV-817S, U11 74HC14 E-stop, U12 AMS1117-3.3, U13 USBLC6-2SC6, U14 USBLC6-2SC6, U15 USBLC6-2SC6, U3 74HC595 #1, U4 74HC595 #2, U5 ULN2803A K1-K8, U6 ULN2803A K9-K16, U7 SN74LVC1G123, U8 74LVC1G00 /OE, U9 74LVC1G11 AND3

Commit message: cook-hub: WIP CHECKPOINT (not a gate) — electrical DRC bucket ELIMINATED (shorts/clearance/mask-bridge 16 -> 0)
Priority-1 fix from ADR-0006 diagnosis: the 6 shorts + 2 clearances + 8
solder-mask-bridges came from decoupler/RC parts pinned directly ONTO IC/
connector pads. Loosened the pins in generate_board.py ANCHOR (all still pass
the IP<=7mm proximity audit), re-routed the full chain:

- watchdog trio out of the U7 pad-field into the free pocket S/E of U7
  (NOGO y<=106.8 forbids N; U8 y117 bounds S): R11->(66.5,114.3) C14->(70,113.5)
  C11->(71.5,110,rot90). IP to U7: 4.3 / 4.95 / 5.0 mm.
- C21 (I2C1 ESD decoupler) was landing pad1 on J2 Pico pad1 (SDA0); moved N of
  its IC U14 -> (30.2,61), IP 3mm.
- U12 (AMS1117) +3mm E -> (56,122): its SOT-223 tab was shorting CE1 GND pad.
- H5 mounting hole (24,62) overlapped connector J4 (mask bridge x2); the west
  edge is fully packed with JST connectors, relocated to the y107-114 gap -> (24,110.5).

GND rescue (stitch_and_fill): added via-in-pad for GND SMD pads (In1 is a solid
GND plane; same-net barrel always bonds a boxed-in pad) + widened the U12 tab
thermal-via search; GND rescue is now non-fatal (DRC unconnected gate catches
genuine misses). Unconnected 64 -> 10.

audit_board I8: D6/R55 added to sanctioned refdes waivers (estop-divider tiny
0603/SOD passives, F.Fab copies, functional net silk nearby — same class as R56).
COST_ESTIMATE + ARCHITECTURE: board size 185x112 -> 185x120 (ADR-0006).

DRC now 480/10/1. NOT a gate: the elevated total vs the inherited 453 is stochastic
KRT route-quality from re-routing from scratch (track_width 45 = 5VP PWR-floor 0.5
thin-passes; via_dangling 32 = 5VP/3V3 F/B vias outside their In2 pours). Remaining
buckets untouched: silk 330 (deterministic), courtyards 44, holes 6, copper-edge 7.
Next: select/tune a clean route + promote (M3), silk de-collision campaign, courtyard
classification, DRU floors to JLC actuals (golden-rule-8).

Co-Authored-By: Claude Fable 5 <noreply@anthropic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
Parts:
- moved TP15 103.5 mm to (176.0, 116.0)
- moved TP16 88.3 mm to (164.0, 124.0)
- moved TP23 80.5 mm to (95.9, 122.4)
- moved C33 80.4 mm to (95.8, 117.4)
- moved R33 78.4 mm to (84.2, 117.4)
- moved TP33 74.2 mm to (132.0, 109.0)
- moved R31 73.8 mm to (86.4, 126.5)
- moved R25 70.0 mm to (128.0, 109.0)
- moved R32 68.9 mm to (90.2, 127.9)
- moved C31 68.7 mm to (90.3, 126.0)
- moved JP5 64.7 mm to (23.9, 116.5)
- moved C9 59.6 mm to (124.0, 109.0)
- moved C17 57.7 mm to (96.0, 120.0)
- moved R34 54.5 mm to (83.9, 113.8)
- moved SJ1 52.0 mm to (55.7, 107.9)
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Routing:
- net 5VP: track 77.2 -> 103.6 mm, vias 6 -> 4
- net VSYS: track 61.7 -> 78.3 mm, vias 0 -> 2
- net 3V3: track 254.6 -> 266.8 mm
- net 3V3A: track 124.5 -> 128.6 mm, vias 2 -> 4
- net 5V_IN: track 10.3 -> 14.0 mm
- net 5V_D: track 8.84 -> 7.84 mm
Other:
- board size 185 x 112 mm -> 185 x 120 mm
- board text added: "/OE"
- board text added: "3V3"
- board text added: "5VP"
- board text added: "E-STOP+DOOR SCHMITT"
- board text added: "ESTOP_OK"
- board text added: "HX CLK"
- board text added: "HX DAT"
- board text added: "RELAY_5V"
- board text added: "TH3_ADC"
- board text added: "WD_OK"

Commit message: cook-hub: WIP CHECKPOINT (not a gate) — mid zone-chamfer + COIL_EN work at 15/2/0; agent hit 529
Co-Authored-By: Claude Fable 5 <noreply@anthropic.com>
Parts:
- moved H6 13.9 mm to (126.0, 124.0)
Routing:
- net 3V3: track 266.8 -> 269.6 mm
- net 5VP: track 103.6 -> 102.7 mm
- net 5V_IN: track 14.0 -> 14.6 mm
Other:
- board text added: "3V3A"
- board text added: "SDA0"
- board text added: "TH1_ADC"
- board text added: "TH2_ADC"
- board text removed: "JP1: I2C0 PU 1-2=2k2 2-3=4k7"
- board text removed: "MAX31865 DNP"

Commit message: cook-hub v1.0 + cook-loadcell v1.0: SEALED releases (2026-07-19)
Both boards sealed at 07_releases/v1.0-2026-07-19/ with sha256 MANIFESTs,
ORDER_READMEs, fab packages (gerbers zip + coded BOM + CPL), pdf sets,
and verification evidence (twin report + renders, DRC gate json,
pin_review.md).

cook-hub v1.0 scoreboard: ERC 0 · parity 0 · DRC severity-all+refill
0/0/0 · AUDIT PASS (I-ISO 6.12mm, 8 slots) · policy FAIL=0 (14P/3W/6H) ·
twin exit 0 (219 checks, 0 unadjudicated criticals) · pin reviews 3/3
PASS · stock 82/82 >= 5x qty5 · render PASS-WITH-NOTES dispositioned.
ORDER_README: §16-condensed bring-up, Pico-2-NOT-included, §1.9 teardown
gate (no appliance hookup until donor keypad facts), §17 open items.

cook-loadcell v1.0 scoreboard: ERC 0 · parity 0 · DRC 0/0/0 (no DRC
waivers) · AUDIT PASS (I-AN 4mm guard) · policy FAIL=0 (8P/4W/7H) · twin
exit 0 (43 checks) · HX711 pin review PASS (E- float ship-blocker fixed;
AVDD 4.30V) · stock PASS · spec §3.7(a-g) mapping recorded in MANIFEST.
BOM well under the $20 target.

Loadcell policy waivers (R-POUR analog-nets, P-POL inline-asserts,
P-KEEP edge-mates, S-VER SS8550) + r0.kicad_pro netclass refresh.
Firmware skeletons (05_firmware: pinmap.h, COBS+CRC32 protocol.h +
PROTOCOL.md, relay_fsm.h fault hierarchy, watchdog.h) ship in-tree.

Co-Authored-By: Claude Fable 5 <noreply@anthropic.com>
Routing:
- net 3V3: track 269.6 -> 283.4 mm, vias 6 -> 7
- net 5VP: track 102.7 -> 103.2 mm, vias 4 -> 6
Other:
- outline, holes or cut-outs redrawn
