File: projects/cook-loadcell/tscircuit/kicad/cook_loadcell.kicad_sch (KiCad schematic)
At the start: 37 parts

Commit message: tscircuit boundary Phase 2: our circuit.json -> annotated kicad_sch converter clears the exporter ceiling
ADR-0001 Phase 1 proved tscircuit AUTHORS our boards node-for-node, but its native
`tsci export -f kicad_sch` has two fidelity-killing bugs: the
Device:U_chip_<footprint> symbol-id collision (2+ many-pin custom-footprint chips
share one symbol and each truncates to 2 pins) and no symbol annotation (netlist
builds 0 nets). This adds OUR own converter from circuit.json's full connectivity
model, bypassing that exporter.

circuit_json_to_kicad_sch.py: each source_component -> a UNIQUE elt:SYM_<refdes>
lib_symbol (collision impossible); each source_port -> a pin keyed to the exact
KiCad pad name (first non-unnamed_* pcb_* port hint; internally-connected duplicate
shields/thermal pads collapse to one pin); nets resolved via
subcircuit_connectivity_map_key + internally_connected propagation; one global_label
per pin as net glue (schwriter2 rule); GND -> ground power symbols + one PWR_FLAG;
no_connect flags for floats; annotated so `kicad-cli sch export netlist` builds real
nets. Coordinates forced to exact 1.27 multiples so pin tips land on their labels.

kicad_sch_parity.py: node-for-node netlist parity gate vs the sealed 04_kicad board
(leading-digit net renames + documented per-board pad-name deltas).

gen_tscircuit.sh: produces kicad/<board>.kicad_sch via the converter (authoritative),
keeps the native export as .native.kicad_sch, runs ERC + the parity gate into
verification/.

GATE (all 3 Phase-1 boards, re-rendered): kicad-cli sch erc --severity-all = 0 errors;
node-for-node parity 0 vs sealed board.
  cook-loadcell           16/16 nets, 75/75 nodes, 2/2 NC
  xt60-usb-supply-rerun   28/28 nets, 151/151 nodes
  esp32-laser-timing      36/36 nets, 189/189 nodes, 25/25 NC
esp32 proof: U1 (ESP32-S3, 41 pads) and J1 (USB-C, 17 distinct pads) truncated to 2
pins each through the native export now export ALL pins and reach parity 0.

Co-Authored-By: Claude Fable 5 <nor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
Parts:
- removed C1, C4, C6: 10uF, symbol Device:capacitor_down
- removed C2, C3, C5, C7: 100nF, symbol Device:capacitor_down
- removed D1, D2: D, symbol Device:diode_down
- removed GND (x8): GND, symbol Custom:rail_down
- removed J1, J2, J3, J4: (no value), symbol Device:U_chip_pinrow3_p2.5mm
- removed J5, J6: (no value), symbol Device:U_chip_pinrow5_p2.5mm
- removed JP1: (no value), symbol Device:U_chip_pinrow3
- removed Q1: (no value), symbol Device:U_chip_sot23
- removed R1: 20kΩ, symbol Device:boxresistor_right
- removed R2: 8.2kΩ, symbol Device:boxresistor_down
- removed R7: 100Ω, symbol Device:boxresistor_down
- removed SJ1: (no value), symbol Device:solderjumper2_down
- removed TP1: TP1, symbol Device:testpoint_right
- removed TP2: TP2, symbol Device:testpoint_right
- removed TP3: TP3, symbol Device:testpoint_right
- removed TP4: TP4, symbol Device:testpoint_right
- removed TP5: TP5, symbol Device:testpoint_right
- removed TP6: TP6, symbol Device:testpoint_right
- removed TP7: TP7, symbol Device:testpoint_right
- removed U1: (no value), symbol Device:U_chip_soic16_p1.27mm
- added C1: 10uF, symbol elt:SYM_C1
- added C2: 100nF, symbol elt:SYM_C2
- added C3: 100nF, symbol elt:SYM_C3
- added C4: 10uF, symbol elt:SYM_C4
- added C5: 100nF, symbol elt:SYM_C5
- added C6: 10uF, symbol elt:SYM_C6
- added C7: 100nF, symbol elt:SYM_C7
- added D1: C5158048, symbol elt:SYM_D1
- added D2: C5158048, symbol elt:SYM_D2
- added J1: C144394, symbol elt:SYM_J1
- added J2: C144394, symbol elt:SYM_J2
- added J3: C144394, symbol elt:SYM_J3
- added J4: C144394, symbol elt:SYM_J4
- added J5: C157991, symbol elt:SYM_J5
- added J6: C157991, symbol elt:SYM_J6
- added JP1: simple_chip, symbol elt:SYM_JP1
- added Q1: C8542, symbol elt:SYM_Q1
- added R1: 20kΩ, symbol elt:SYM_R1
- added R2: 8.2kΩ, symbol elt:SYM_R2
- added R7: 100Ω, symbol elt:SYM_R7
- added SJ1: simple_chip, symbol elt:SYM_SJ1
- added TP1: simple_test_point, symbol elt:SYM_TP1
- added TP2: simple_test_point, symbol elt:SYM_TP2
- added TP3: simple_test_point, symbol elt:SYM_TP3
- added TP4: simple_test_point, symbol elt:SYM_TP4
- added TP5: simple_test_point, symbol elt:SYM_TP5
- added TP6: simple_test_point, symbol elt:SYM_TP6
- added TP7: simple_test_point, symbol elt:SYM_TP7
- added U1: C43656, symbol elt:SYM_U1
Connections:
- net AVDD_FB: now also R1.2 (pin2), R2.1 (pin1), U1.4 (VFB)
- net BASE: now also Q1.1 (B), U1.2 (BASE)
- net CLK: now also D2.1 (pin1), J6.5 (pin5), TP6.1 (pin1), U1.11 (PD_SCK)
- net DAT: now also D1.1 (pin1), J6.4 (pin4), TP5.1 (pin1), U1.12 (DOUT)
- net E_PLUS: now also C1.1 (pin1), C2.1 (pin1), J1.2 (pin2), J5.1 (pin1), Q1.3 (C), R1.1 (pin1), TP1.1 (pin1), U1.3 (AVDD)
- net GND: now also C1.2 (pin2), C2.2 (pin2), C3.2 (pin2), C4.2 (pin2), C5.2 (pin2), C6.2 (pin2), C7.2 (pin2), D1.2 (pin2), D2.2 (pin2), J3.2 (pin2), J5.4 (pin4), J6.3 (pin3), JP1.1 (pin1), R2.2 (pin2), R7.2 (pin2), SJ1.2 (pin2), TP4.1 (pin1), U1.10 (INB_P), U1.14 (XI), U1.5 (AGND), U1.9 (INB_N)
- net N3V3: now also C3.1 (pin1), C4.1 (pin1), J6.2 (pin2), JP1.3 (pin3), TP7.1 (pin1), U1.16 (DVDD)
- net N5V: now also C5.1 (pin1), C6.1 (pin1), J6.1 (pin1), Q1.2 (E), U1.1 (VSUP)
- net RATE_SEL: now also JP1.2 (pin2), U1.15 (RATE)
- net RING_12: now also J1.3 (pin3), J2.1 (pin1)
- net RING_23: now also J2.3 (pin3), J3.1 (pin1)
- net RING_34: now also J3.3 (pin3), J4.1 (pin1)
- net RING_41: now also J1.1 (pin1), J4.3 (pin3)
- net SH: now also C7.1 (pin1), J5.5 (pin5), R7.1 (pin1), SJ1.1 (pin1)
- net S_MINUS: now also J4.2 (pin2), J5.3 (pin3), TP3.1 (pin1), U1.7 (INA_N)
- net S_PLUS: now also J2.2 (pin2), J5.2 (pin2), TP2.1 (pin1), U1.8 (INA_P)
- no-connect marks 0 -> 2
Other:
- title: (none) -> cook_loadcell

Commit message: tscircuit backend completion (ADR-0001): fold Phase-3 adapter INTO the converter — output is backend-ready, no per-board adapter
The Phase-3 proof reached DRC 0/0/0 only via a one-shot project-local adapter
(prepare_backend_sch.py + assign_footprints.py) that patched five converter gaps.
Fold gaps 1-4 into circuit_json_to_kicad_sch.py so the converter output feeds the
full KiCad backend directly:

1. Canonical net names: canon_net strips a documented author-prefix `N` guarding a
   digit-leading rail (N5V->5V, N3V3->3V3, N5V_A->5V_A; NRST/NC untouched) + an
   optional auto-discovered per-board tscircuit/net_aliases.txt for the rest.
2. Footprint FPIDs: baked-in commodity token->FPID map (circuit.json's
   cad_component.footprinter_string class-disambiguates res0603 vs 0603) + a
   per-board override auto-seeded from 02_parts/*/part.yaml (LCSC/JLC/MPN/folder ->
   footprint), which wins for specialty parts. part.yaml footprint read as first
   whitespace-free token so a trailing YAML `# comment` (TS-1187A, with quotes)
   can't corrupt the s-expr.
3. Drop the MPN symbol field (footprint_symbol_field_mismatch).
4. Test points: in_bom no + concise `TP` value (no board-edge silk clip).

GATE RESULTS:
A. All 3 ladder boards, converter -> ERC 0 + netlist parity 0 (unchanged from
   Phase 2): cook-loadcell 16/75, xt60 28/151, esp32 36/189.
B. cook-loadcell full backend from the converter output ALONE (build_from_tsx.sh
   step [1] is now a plain cp, adapters bypassed): generate_board -> rules -> KRT
   -> stitch -> DRC --severity-all --refill-zones --schematic-parity = 0/0/0, and
   board-netlist parity 0 vs the sealed board (77/77 nodes, 17/17 nets).
C. xt60 + esp32 emit canonical nets + FPIDs + TP BOM attrs too (esp32 72/72 FPID
   incl. specialty from 02_parts; xt60 34/47 — the 13 gaps are hand-<footprint>
   specialty parts whose TSX omits supplierPartNumbers).

prepare_backend_sch.py / assign_footprints.py marked SUPERSEDED (kept for record);
NOTES.md + ADR-0001 back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
Parts:
- C1, C4, C6: footprint (none) -> Capacitor_SMD:C_0805_2012Metric; MPN C15850 -> (none)
- C2, C3, C5, C7: footprint (none) -> Capacitor_SMD:C_0603_1608Metric; MPN C14663 -> (none)
- D1, D2: footprint (none) -> Diode_SMD:D_SOD-323; MPN C5158048 -> (none)
- J1, J2, J3, J4: footprint (none) -> Connector_JST:JST_XH_B3B-XH-A_1x03_P2.50mm_Vertical; MPN C144394 -> (none)
- J5, J6: footprint (none) -> Connector_JST:JST_XH_B5B-XH-A_1x05_P2.50mm_Vertical; MPN C157991 -> (none)
- JP1: footprint (none) -> Connector_PinHeader_2.54mm:PinHeader_1x03_P2.54mm_Vertical
- Q1: footprint (none) -> Package_TO_SOT_SMD:SOT-23; MPN C8542 -> (none)
- R1: footprint (none) -> Resistor_SMD:R_0603_1608Metric; MPN C4184 -> (none)
- R2: footprint (none) -> Resistor_SMD:R_0603_1608Metric; MPN C25981 -> (none)
- R7: footprint (none) -> Resistor_SMD:R_0603_1608Metric; MPN C22775 -> (none)
- SJ1: footprint (none) -> Jumper:SolderJumper-2_P1.3mm_Open_Pad1.0x1.5mm
- TP1, TP2, TP3, TP4, TP5, TP6, TP7: value simple_test_point -> TP; footprint (none) -> TestPoint:TestPoint_Pad_D1.5mm; now left out of the parts list
- U1: footprint (none) -> Package_SO:SOIC-16_3.9x9.9mm_P1.27mm; MPN C43656 -> (none)
Connections:
- net N3V3 renamed 3V3
- net N5V renamed 5V
