File: projects/esp32-laser-timing/tscircuit/kicad/esp32_laser_timing.kicad_sch (KiCad schematic)
At the start: 97 parts, among them SW1 SW1, SW2 SW2

Commit message: tscircuit boundary Phase 2: our circuit.json -> annotated kicad_sch converter clears the exporter ceiling
ADR-0001 Phase 1 proved tscircuit AUTHORS our boards node-for-node, but its native
`tsci export -f kicad_sch` has two fidelity-killing bugs: the
Device:U_chip_<footprint> symbol-id collision (2+ many-pin custom-footprint chips
share one symbol and each truncates to 2 pins) and no symbol annotation (netlist
builds 0 nets). This adds OUR own converter from circuit.json's full connectivity
model, bypassing that exporter.

circuit_json_to_kicad_sch.py: each source_component -> a UNIQUE elt:SYM_<refdes>
lib_symbol (collision impossible); each source_port -> a pin keyed to the exact
KiCad pad name (first non-unnamed_* pcb_* port hint; internally-connected duplicate
shields/thermal pads collapse to one pin); nets resolved via
subcircuit_connectivity_map_key + internally_connected propagation; one global_label
per pin as net glue (schwriter2 rule); GND -> ground power symbols + one PWR_FLAG;
no_connect flags for floats; annotated so `kicad-cli sch export netlist` builds real
nets. Coordinates forced to exact 1.27 multiples so pin tips land on their labels.

kicad_sch_parity.py: node-for-node netlist parity gate vs the sealed 04_kicad board
(leading-digit net renames + documented per-board pad-name deltas).

gen_tscircuit.sh: produces kicad/<board>.kicad_sch via the converter (authoritative),
keeps the native export as .native.kicad_sch, runs ERC + the parity gate into
verification/.

GATE (all 3 Phase-1 boards, re-rendered): kicad-cli sch erc --severity-all = 0 errors;
node-for-node parity 0 vs sealed board.
  cook-loadcell           16/16 nets, 75/75 nodes, 2/2 NC
  xt60-usb-supply-rerun   28/28 nets, 151/151 nodes
  esp32-laser-timing      36/36 nets, 189/189 nodes, 25/25 NC
esp32 proof: U1 (ESP32-S3, 41 pads) and J1 (USB-C, 17 distinct pads) truncated to 2
pins each through the native export now export ALL pins and reach parity 0.

Co-Authored-By: Claude Fable 5 <nor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
Parts:
- removed C1: 1uF, symbol Device:capacitor_down
- removed C10, C12, C5, C6, C7, C8, C9: 100nF, symbol Device:capacitor_down
- removed C11: 100uF, symbol Device:capacitor_polarized_down
- removed C2, C3, C4: 22uF, symbol Device:capacitor_down
- removed D1: (no value), symbol Device:U_chip_sot23_6
- removed D2: (no value), symbol Device:led_up
- removed GND (x22): GND, symbol Custom:rail_down
- removed J1, J10, J11, J12, J4, J5, J6, J7, J8, J9, U1: (no value), symbol Device:U_chip
- removed J2: (no value), symbol Device:U_chip_pinrow4
- removed Q1, Q2, Q3: (no value), symbol Device:U_chip_sot23
- removed R1, R2: 5.1kΩ, symbol Device:boxresistor_down
- removed R10, R12, R14: 100Ω, symbol Device:boxresistor_right
- removed R11, R13, R15: 100kΩ, symbol Device:boxresistor_down
- removed R20, R21, R22: 1kΩ, symbol Device:boxresistor_down
- removed R23, R24, R25: 10kΩ, symbol Device:boxresistor_up
- removed R26, R27, R28: 2.7kΩ, symbol Device:boxresistor_down
- removed R29, R30, R31: 33kΩ, symbol Device:boxresistor_right
- removed R3, R32, R33, R34, R40, R41, R42: 10kΩ, symbol Device:boxresistor_right
- removed R4, R43, R44, R45: 1kΩ, symbol Device:boxresistor_right
- removed R50, R51: 4.7kΩ, symbol Device:boxresistor_right
- removed SW1: SW1, symbol Device:push_button_normally_open_momentary_down
- removed SW2: SW2, symbol Device:push_button_normally_open_momentary_down
- removed TP1: TP1, symbol Device:testpoint_right
- removed TP2: TP2, symbol Device:testpoint_right
- removed TP3: TP3, symbol Device:testpoint_right
- removed TP4: TP4, symbol Device:testpoint_right
- removed TP5: TP5, symbol Device:testpoint_right
- removed TP6: TP6, symbol Device:testpoint_right
- removed U2: (no value), symbol Device:U_chip_sot223
- removed U3: (no value), symbol Device:U_chip_soic14_p1.27mm
- removed VTH1: VTH1, symbol Custom:rail_up
- removed VTH2 (x2): VTH2, symbol Custom:rail_up
- added C1: 1uF, symbol elt:SYM_C1
- added C10: 100nF, symbol elt:SYM_C10
- added C11: 100uF, symbol elt:SYM_C11
- added C12: 100nF, symbol elt:SYM_C12
- added C2: 22uF, symbol elt:SYM_C2
- added C3: 22uF, symbol elt:SYM_C3
- added C4: 22uF, symbol elt:SYM_C4
- added C5: 100nF, symbol elt:SYM_C5
- added C6: 100nF, symbol elt:SYM_C6
- added C7: 100nF, symbol elt:SYM_C7
- added C8: 100nF, symbol elt:SYM_C8
- added C9: 100nF, symbol elt:SYM_C9
- added D1: C2687116, symbol elt:SYM_D1
- added D2: C2297, symbol elt:SYM_D2
- added J1: C165948, symbol elt:SYM_J1
- added J10: C474930, symbol elt:SYM_J10
- added J11: C474930, symbol elt:SYM_J11
- added J12: C474930, symbol elt:SYM_J12
- added J2: C2718488, symbol elt:SYM_J2
- added J4: C474930, symbol elt:SYM_J4
- added J5: C474930, symbol elt:SYM_J5
- added J6: C474930, symbol elt:SYM_J6
- added J7: C474930, symbol elt:SYM_J7
- added J8: C474930, symbol elt:SYM_J8
- added J9: C474930, symbol elt:SYM_J9
- added Q1: C20917, symbol elt:SYM_Q1
- added Q2: C20917, symbol elt:SYM_Q2
- added Q3: C20917, symbol elt:SYM_Q3
- added R1: 5.1kΩ, symbol elt:SYM_R1
- added R10: 100Ω, symbol elt:SYM_R10
- added R11: 100kΩ, symbol elt:SYM_R11
- added R12: 100Ω, symbol elt:SYM_R12
- added R13: 100kΩ, symbol elt:SYM_R13
- added R14: 100Ω, symbol elt:SYM_R14
- added R15: 100kΩ, symbol elt:SYM_R15
- added R2: 5.1kΩ, symbol elt:SYM_R2
- added R20: 1kΩ, symbol elt:SYM_R20
- added R21: 1kΩ, symbol elt:SYM_R21
- added R22: 1kΩ, symbol elt:SYM_R22
- added R23: 10kΩ, symbol elt:SYM_R23
- added R24: 10kΩ, symbol elt:SYM_R24
- added R25: 10kΩ, symbol elt:SYM_R25
- added R26: 2.7kΩ, symbol elt:SYM_R26
- added R27: 2.7kΩ, symbol elt:SYM_R27
- added R28: 2.7kΩ, symbol elt:SYM_R28
- added R29: 33kΩ, symbol elt:SYM_R29
- added R3: 10kΩ, symbol elt:SYM_R3
- added R30: 33kΩ, symbol elt:SYM_R30
- added R31: 33kΩ, symbol elt:SYM_R31
- added R32: 10kΩ, symbol elt:SYM_R32
- added R33: 10kΩ, symbol elt:SYM_R33
- added R34: 10kΩ, symbol elt:SYM_R34
- added R4: 1kΩ, symbol elt:SYM_R4
- added R40: 10kΩ, symbol elt:SYM_R40
- added R41: 10kΩ, symbol elt:SYM_R41
- added R42: 10kΩ, symbol elt:SYM_R42
- added R43: 1kΩ, symbol elt:SYM_R43
- added R44: 1kΩ, symbol elt:SYM_R44
- added R45: 1kΩ, symbol elt:SYM_R45
- added R50: 4.7kΩ, symbol elt:SYM_R50
- added R51: 4.7kΩ, symbol elt:SYM_R51
- added SW1: C318884, symbol elt:SYM_SW1
- added SW2: C318884, symbol elt:SYM_SW2
- added TP1: simple_test_point, symbol elt:SYM_TP1
- added TP2: simple_test_point, symbol elt:SYM_TP2
- added TP3: simple_test_point, symbol elt:SYM_TP3
- added TP4: simple_test_point, symbol elt:SYM_TP4
- added TP5: simple_test_point, symbol elt:SYM_TP5
- added TP6: simple_test_point, symbol elt:SYM_TP6
- added U1: C2913204, symbol elt:SYM_U1
- added U2: C6186, symbol elt:SYM_U2
- added U3: C71036, symbol elt:SYM_U3
Connections:
- net BOOT: now also SW1.1 (pin1), U1.27 (IO0)
- net BTN1_G: now also R43.2 (pin2), U1.10 (IO17)
- net BTN1_N: now also C8.1 (pin1), J10.1 (pin1), R40.2 (pin2), R43.1 (pin1)
- net BTN2_G: now also R44.2 (pin2), U1.11 (IO18)
- net BTN2_N: now also C9.1 (pin1), J11.1 (pin1), R41.2 (pin2), R44.1 (pin1)
- net BTN3_G: now also R45.2 (pin2), U1.23 (IO21)
- net BTN3_N: now also C10.1 (pin1), J12.1 (pin1), R42.2 (pin2), R45.1 (pin1)
- net CC1: now also J1.A5 (pin3), R1.1 (pin1)
- net CC2: now also J1.B5 (pin11), R2.1 (pin1)
- net COMP1: now also R29.2 (pin2), R32.2 (pin2), TP1.1 (pin1), U1.4 (IO4), U3.2 (OUT1)
- net COMP2: now also R30.2 (pin2), R33.2 (pin2), TP2.1 (pin1), U1.5 (IO5), U3.1 (OUT2)
- net COMP3: now also R31.2 (pin2), R34.2 (pin2), TP3.1 (pin1), U1.6 (IO6), U3.14 (OUT3)
- net EN: now also C1.1 (pin1), R3.2 (pin2), SW2.1 (pin1), U1.3 (EN)
- net GATE1: now also Q1.1 (G), R10.2 (pin2), R11.1 (pin1)
- net GATE2: now also Q2.1 (G), R12.2 (pin2), R13.1 (pin1)
- net GATE3: now also Q3.1 (G), R14.2 (pin2), R15.1 (pin1)
- net LDRV1: now also R10.1 (pin1), U1.7 (IO7)
- net LDRV2: now also R12.1 (pin1), U1.8 (IO15)
- net LDRV3: now also R14.1 (pin1), U1.9 (IO16)
- net LED_A: now also D2.2 (pin2), R4.2 (pin2)
- net LSW1: now also J4.2 (pin2), Q1.3 (D)
- net LSW2: now also J5.2 (pin2), Q2.3 (D)
- net LSW3: now also J6.2 (pin2), Q3.3 (D)
- net N3V3: now also C3.1 (pin1), C4.1 (pin1), C5.1 (pin1), C7.1 (pin1), J2.2 (pin2), R23.1 (pin1), R24.1 (pin1), R25.1 (pin1), R3.1 (pin1), R32.1 (pin1), R33.1 (pin1), R34.1 (pin1), R4.1 (pin1), R40.1 (pin1), R41.1 (pin1), R42.1 (pin1), R50.1 (pin1), R51.1 (pin1), TP5.1 (pin1), U1.2 (V3V3), U2.2 (VOUT), U2.4 (TAB)
- net N5V: now also C11.1 (pin1), C12.1 (pin1), C2.1 (pin1), C6.1 (pin1), D1.5 (VBUS), J1.A4 (pin2), J1.A9 (pin7), J1.B4 (pin10), J1.B9 (pin15), J4.1 (pin1), J5.1 (pin1), J6.1 (pin1), J7.1 (pin1), J8.1 (pin1), J9.1 (pin1), TP4.1 (pin1), U2.3 (VIN), U3.3 (VCC)
- net PD1: now also J7.2 (pin2), R20.1 (pin1), R29.1 (pin1), U3.5 (IN1p)
- net PD2: now also J8.2 (pin2), R21.1 (pin1), R30.1 (pin1), U3.7 (IN2p)
- net PD3: now also J9.2 (pin2), R22.1 (pin1), R31.1 (pin1), U3.9 (IN3p)
- net SCL: now also J2.3 (pin3), R51.2 (pin2), U1.38 (IO2)
- net SDA: now also J2.4 (pin4), R50.2 (pin2), U1.39 (IO1)
- net USB_DM: now also D1.3 (IO2), D1.4 (IO2b), J1.A7 (pin5), J1.B7 (pin13), U1.13 (IO19_DM)
- net USB_DP: now also D1.1 (IO1), D1.6 (IO1b), J1.A6 (pin4), J1.B6 (pin12), U1.14 (IO20_DP)
- net VTH1: now also R23.2 (pin2), R26.1 (pin1), U3.4 (IN1n)
- net VTH3: now also R25.2 (pin2), R28.1 (pin1), U3.10 (IN4n), U3.8 (IN3n)
- new net GND: C1.2 (pin2), C10.2 (pin2), C11.2 (pin2), C12.2 (pin2), C2.2 (pin2), C3.2 (pin2), C4.2 (pin2), C5.2 (pin2), C6.2 (pin2), C7.2 (pin2), C8.2 (pin2), C9.2 (pin2), D1.2 (GND), D2.1 (pin1), J1.A1 (pin1), J1.A12 (pin8), J1.B1 (pin9), J1.B12 (pin16), J1.SH (pin17), J10.2 (pin2), J11.2 (pin2), J12.2 (pin2), J2.1 (pin1), Q1.2 (S), Q2.2 (S), Q3.2 (S), R1.2 (pin2), R11.2 (pin2), R13.2 (pin2), R15.2 (pin2), R2.2 (pin2), R20.2 (pin2), R21.2 (pin2), R22.2 (pin2), R26.2 (pin2), R27.2 (pin2), R28.2 (pin2), SW1.2 (pin2), SW2.2 (pin2), TP6.1 (pin1), U1.1 (GND), U1.40 (GND40), U1.41 (EPAD), U2.1 (GND), U3.11 (IN4p), U3.12 (GND)
- new net VTH2: R24.2 (pin2), R27.1 (pin1), U3.6 (IN2n)
- no-connect marks 0 -> 25
Other:
- title: (none) -> esp32_laser_timing

Commit message: tscircuit backend completion (ADR-0001): fold Phase-3 adapter INTO the converter — output is backend-ready, no per-board adapter
The Phase-3 proof reached DRC 0/0/0 only via a one-shot project-local adapter
(prepare_backend_sch.py + assign_footprints.py) that patched five converter gaps.
Fold gaps 1-4 into circuit_json_to_kicad_sch.py so the converter output feeds the
full KiCad backend directly:

1. Canonical net names: canon_net strips a documented author-prefix `N` guarding a
   digit-leading rail (N5V->5V, N3V3->3V3, N5V_A->5V_A; NRST/NC untouched) + an
   optional auto-discovered per-board tscircuit/net_aliases.txt for the rest.
2. Footprint FPIDs: baked-in commodity token->FPID map (circuit.json's
   cad_component.footprinter_string class-disambiguates res0603 vs 0603) + a
   per-board override auto-seeded from 02_parts/*/part.yaml (LCSC/JLC/MPN/folder ->
   footprint), which wins for specialty parts. part.yaml footprint read as first
   whitespace-free token so a trailing YAML `# comment` (TS-1187A, with quotes)
   can't corrupt the s-expr.
3. Drop the MPN symbol field (footprint_symbol_field_mismatch).
4. Test points: in_bom no + concise `TP` value (no board-edge silk clip).

GATE RESULTS:
A. All 3 ladder boards, converter -> ERC 0 + netlist parity 0 (unchanged from
   Phase 2): cook-loadcell 16/75, xt60 28/151, esp32 36/189.
B. cook-loadcell full backend from the converter output ALONE (build_from_tsx.sh
   step [1] is now a plain cp, adapters bypassed): generate_board -> rules -> KRT
   -> stitch -> DRC --severity-all --refill-zones --schematic-parity = 0/0/0, and
   board-netlist parity 0 vs the sealed board (77/77 nodes, 17/17 nets).
C. xt60 + esp32 emit canonical nets + FPIDs + TP BOM attrs too (esp32 72/72 FPID
   incl. specialty from 02_parts; xt60 34/47 — the 13 gaps are hand-<footprint>
   specialty parts whose TSX omits supplierPartNumbers).

prepare_backend_sch.py / assign_footprints.py marked SUPERSEDED (kept for record);
NOTES.md + ADR-0001 back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
Parts:
- C1: footprint (none) -> Capacitor_SMD:C_0805_2012Metric; MPN C28323 -> (none)
- C10, C12, C5, C6, C7, C8, C9: footprint (none) -> Capacitor_SMD:C_0805_2012Metric; MPN C49678 -> (none)
- C11: footprint (none) -> Capacitor_SMD:CP_Elec_6.3x5.4; MPN C2887276 -> (none)
- C2, C3, C4: footprint (none) -> Capacitor_SMD:C_0805_2012Metric; MPN C45783 -> (none)
- D1: footprint (none) -> Package_TO_SOT_SMD:SOT-23-6; MPN C2687116 -> (none)
- D2: footprint (none) -> LED_SMD:LED_0805_2012Metric; MPN C2297 -> (none)
- J1: footprint (none) -> Connector_USB:USB_C_Receptacle_HRO_TYPE-C-31-M-12; MPN C165948 -> (none)
- J10, J11, J12, J4, J5, J6, J7, J8, J9: footprint (none) -> TerminalBlock_Phoenix:TerminalBlock_Phoenix_PT-1,5-2-3.5-H_1x02_P3.50mm_Horizontal; MPN C474930 -> (none)
- J2: footprint (none) -> Connector_PinSocket_2.54mm:PinSocket_1x04_P2.54mm_Vertical; MPN C2718488 -> (none)
- Q1, Q2, Q3: footprint (none) -> Package_TO_SOT_SMD:SOT-23; MPN C20917 -> (none)
- R1, R2: footprint (none) -> Resistor_SMD:R_0805_2012Metric; MPN C27834 -> (none)
- R10, R12, R14: footprint (none) -> Resistor_SMD:R_0805_2012Metric; MPN C17408 -> (none)
- R11, R13, R15: footprint (none) -> Resistor_SMD:R_0805_2012Metric; MPN C149504 -> (none)
- R20, R21, R22, R4, R43, R44, R45: footprint (none) -> Resistor_SMD:R_0805_2012Metric; MPN C17513 -> (none)
- R23, R24, R25, R3, R32, R33, R34, R40, R41, R42: footprint (none) -> Resistor_SMD:R_0805_2012Metric; MPN C17414 -> (none)
- R26, R27, R28: footprint (none) -> Resistor_SMD:R_0805_2012Metric; MPN C17530 -> (none)
- R29, R30, R31: footprint (none) -> Resistor_SMD:R_0805_2012Metric; MPN C17633 -> (none)
- R50, R51: footprint (none) -> Resistor_SMD:R_0805_2012Metric; MPN C17673 -> (none)
- SW1, SW2: footprint (none) -> Button_Switch_SMD:SW_Push_1P1T_XKB_TS-1187A; MPN C318884 -> (none)
- TP1, TP2, TP3, TP4, TP5, TP6: value simple_test_point -> TP; footprint (none) -> TestPoint:TestPoint_Pad_D1.5mm; now left out of the parts list
- U1: footprint (none) -> esp32_laser_timing:ESP32-S3-WROOM-1; MPN C2913204 -> (none)
- U2: footprint (none) -> Package_TO_SOT_SMD:SOT-223-3_TabPin2; MPN C6186 -> (none)
- U3: footprint (none) -> Package_SO:SOIC-14_3.9x8.7mm_P1.27mm; MPN C71036 -> (none)
Connections:
- net N3V3 renamed 3V3
- net N5V renamed 5V
