File: projects/usb-hub-3s/04_kicad/usb_hub_3s.kicad_pcb (KiCad board)
At the start: 4 copper layers, 110 x 90 mm, 116 parts, among them J1 C98732, J2 C503996, J3 C503996, J4 C503996, J5 C5337088, Q1 C2760089, Q10 C8545, Q11 C15127, Q12 C8545, Q2 C404363, Q3 C404363, Q4 C404363, Q5 C404363, Q6 C404363, Q7 C404363, Q8 C404363, Q9 C15127, U1 C5140592, U10 C7519, U2 C13755, U3 C130056, U4 C130056, U5 C130056, U6 C473910, U7 C473910, U8 C7519, U9 C7519

Commit message: usb-hub-3s v1.1 WIP: placement green (audit PASS, 0 courtyard overlaps) + route iterations 1-3 journaled
Board regenerated from the re-floorplanned cell; measured adjacencies:
HS-LS edge gaps 1.4/1.6mm, C46->Q4.D 2.85mm, kelvin stubs 3.3-5.8mm,
gate-Rs 2.8-4.3mm. Route runs 1-3: 0 copper violations each; tap-threading
of the four long chip-pin pour connections proved fragile (KRT hugs lane
edges) -> deterministic seed stubs (add_seed_stubs.py + seed_stubs.yaml)
with crossing-gap corridors; VCC5V/VCCIO promoted to the emk wave after
measured sig-wave starvation. Route 4 in flight.

Co-Authored-By: Claude Fable 5 <noreply@anthropic.com>
Parts:
- added C44: C2982822, Capacitor_SMD:CP_Elec_6.3x7.7, F.Cu at (89.5, 61.0)
- added C45: 10uF, Capacitor_SMD:C_1210_3225Metric, F.Cu at (89.4, 68.3)
- added C46: 10uF, Capacitor_SMD:C_1210_3225Metric, F.Cu at (78.8, 67.7)
- added C47: 10uF, Capacitor_SMD:C_1210_3225Metric, F.Cu at (82.3, 67.7)
- added C48: 100nF, Capacitor_SMD:C_0603_1608Metric, F.Cu at (82.5, 64.4)
- added C49: 10uF, Capacitor_SMD:C_1210_3225Metric, F.Cu at (45.4, 71.1)
- added C50: 10uF, Capacitor_SMD:C_1210_3225Metric, F.Cu at (45.4, 74.7)
- added C51: 100nF, Capacitor_SMD:C_0603_1608Metric, F.Cu at (44.8, 68.6)
- added R28: 0Ω, Resistor_SMD:R_0603_1608Metric, F.Cu at (79.4, 77.7)
- added R29: 0Ω, Resistor_SMD:R_0603_1608Metric, F.Cu at (70.0, 69.3)
- added R30: 0Ω, Resistor_SMD:R_0603_1608Metric, F.Cu at (56.3, 69.3)
- added R31: 0Ω, Resistor_SMD:R_0603_1608Metric, F.Cu at (62.6, 68.5)
- D6: value C148230 -> C148216
- D7: value C148230 -> C148222
- L1: value C5240401 -> C20613209; footprint Inductor_SMD:L_Sunlord_MWSA1707S -> usb_hub_3s:L_YJYCOIN_YSPI1770Y
- Q4, Q5, Q6, Q7, Q8: value C404363 -> C431185
- moved R19 24.7 mm to (44.2, 82.6)
- moved R18 23.8 mm to (44.0, 78.2)
- moved D1 20.3 mm to (41.0, 105.0)
- moved R14 19.7 mm to (89.3, 77.5), turned to -90 degrees
- moved C2 19.5 mm to (38.4, 97.8), turned to 90 degrees
- moved C1 17.7 mm to (38.4, 88.0), turned to 90 degrees
- moved C23 14.8 mm to (77.0, 84.6), turned to 90 degrees
- moved L1 11.5 mm to (65.5, 85.6)
- moved Q5 11.3 mm to (71.0, 73.0)
- moved Q7 11.0 mm to (60.0, 73.0)
- moved R16 10.9 mm to (77.0, 80.9), turned to -90 degrees
- moved R15 10.5 mm to (83.3, 78.4), turned to -90 degrees
- moved C27 9.14 mm to (54.3, 88.6), turned to 90 degrees
- moved C22 9.10 mm to (66.8, 69.2)
- moved RS3 9.01 mm to (47.5, 80.5)
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Connections:
- D1 pad 1: VBAT_F -> VIN
- Q4 pad 4: HG2 -> QG4
- Q5 pad 4: LG2 -> QG5
- Q6 pad 4: HG1 -> QG6
- Q7 pad 4: LG1 -> QG7
Routing:
- net 5VA: track 108.6 -> 0.00 mm, vias 8 -> 0
- net DMC: track 91.3 -> 0.00 mm, vias 5 -> 0
- net CC2: track 79.4 -> 0.00 mm, vias 6 -> 0
- net DPC: track 76.4 -> 0.00 mm, vias 5 -> 0
- net CC1: track 73.4 -> 0.00 mm, vias 6 -> 0
- net EMK1: track 73.1 -> 0.00 mm, vias 2 -> 0
- net EMK2: track 72.1 -> 0.00 mm, vias 2 -> 0
- net EN_PD: track 51.5 -> 0.00 mm, vias 2 -> 0
- net VOUT2_SNS: track 48.6 -> 0.00 mm
- net PATH_G: track 45.7 -> 0.00 mm
- net DP_A2: track 44.2 -> 0.00 mm
- net DM_A2: track 42.3 -> 0.00 mm
- net DP_A3: track 39.7 -> 0.00 mm
- net VOUT_PD: track 39.4 -> 0.00 mm, vias 5 -> 0
- net VCONN5V: track 38.7 -> 0.00 mm, vias 11 -> 0
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- removed copper zone on B.Cu, net LX1
- removed copper zone on B.Cu, net LX2
Other:
- board text added: "C44"
- board text added: "C45"
- board text added: "C46"
- board text added: "C47"
- board text added: "C48"
- board text added: "C49"
- board text added: "C50"
- board text added: "C51"
- board text added: "ONLY - 9-12.6V IN"
- board text added: "PROTECTED 3S PACK"
- board text added: "R28"
- board text added: "R29"
- board text added: "R30"
- board text added: "R31"
- board text added: "usb-hub-3s v1.1"
- board text removed: "3S LIPO 9-12.6V"
- board text removed: "usb-hub-3s v1.0"
