File: projects/usb-hub-3s/04_kicad/usb_hub_3s.kicad_pcb (KiCad board)
At the start: 4 copper layers, 110 x 90 mm, 128 parts, among them J1 C98732, J2 C503996, J3 C503996, J4 C503996, J5 C5337088, Q1 C2760089, Q10 C8545, Q11 C15127, Q12 C8545, Q2 C404363, Q3 C404363, Q4 C431185, Q5 C431185, Q6 C431185, Q7 C431185, Q8 C431185, Q9 C15127, U1 C5140592, U10 C7519, U2 C13755, U3 C130056, U4 C130056, U5 C130056, U6 C473910, U7 C473910, U8 C7519, U9 C7519

Commit message: usb-hub-3s v1.1 WIP checkpoint: PD-cell re-layout mid-grind (session-limit interrupt) — floorplan/route/board + DETAIL_DESIGN + routing journal preserved; route clean per agent (7 tap-owned J5 opens) with 3 zones-intersect defects pending; interim raw DRC 15v/84u reflects unfilled pours mid-surgery, NOT a regression
Parts:
- moved C22 6.46 mm to (60.6, 67.4), turned to -90 degrees
- moved R29 6.23 mm to (66.5, 74.5), turned to -90 degrees
- moved C21 2.60 mm to (70.6, 69.2)
- moved R17 1.90 mm to (57.7, 69.3)
- moved R30 1.80 mm to (54.5, 69.3)
- turned R31 to -90 degrees
Routing:
- net DPC: track 0.00 -> 102.8 mm, vias 0 -> 6
- net 5VA: track 0.00 -> 95.1 mm, vias 0 -> 4
- net DMC: track 0.00 -> 89.8 mm, vias 0 -> 6
- net CC1: track 0.00 -> 83.4 mm, vias 0 -> 8
- net CC2: track 0.00 -> 77.0 mm, vias 0 -> 8
- net EMK1: track 0.00 -> 73.0 mm, vias 0 -> 2
- net EMK2: track 0.00 -> 71.2 mm, vias 0 -> 4
- net VOUT2_SNS: track 0.00 -> 63.2 mm, vias 0 -> 2
- net BST1: track 0.00 -> 63.1 mm, vias 0 -> 2
- net EN_PD: track 0.00 -> 59.4 mm, vias 0 -> 7
- net PATH_G: track 0.00 -> 59.0 mm, vias 0 -> 2
- net SNS_OUT_P: track 0.00 -> 52.5 mm, vias 0 -> 2
- net HG1: track 0.00 -> 47.4 mm, vias 0 -> 8
- net DP_A2: track 0.00 -> 47.1 mm
- net SNS_IN_P: track 0.00 -> 41.9 mm, vias 0 -> 4
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
Commit message: usb-hub-3s v1.1: checkpoint loose working-tree (route.yaml/final_chain/circuit.json) from the stopped Opus finish agent before the Haiku grind resume
Routing:
- net VOUT_PDS: vias 6 -> 0
- net VOUT_PD: vias 8 -> 2
- net VIN_S: vias 6 -> 0
- net VIN: vias 8 -> 2
- net VBAT_F: vias 6 -> 0
- net SW_A: vias 8 -> 2
- net GND: vias 16 -> 8
