File: projects/crow-mic-pod-v2/03_src/route/r3.kicad_pcb (KiCad board)
At the start: 2 copper layers, 80 x 45 mm, 39 parts, among them J1 C9900035627, U1 C192421

Commit message: crow-mic-pod-v2: verification checkpoint — 4-lens red-team, DO NOT ORDER (3 P0)
Banks the red-team evidence + the reproducibility fix before the fix pass (WIP: a
failed/blocked state is evidence, not a release). Board is DRC 0/0/0 / parity 0 and the
documented pinout + 3 V/V gain are internally correct, but the 4 zero-context lenses
(08_reviews/ + DISPOSITIONS.md) found 3 P0 seal-blockers:
- A/B PoE power injection: 5V_AUDIO aliases onto PoE Alt-B, drives 44-57V into OPA1678
  V+ (40V max) -> U1 destroyed. Root: RJ45-everywhere (ADR-0003) + protection-delegation
  (ADR-0001), neither analyzed power injection. USER DECISION: accept with documented
  sign-off (controlled deployment, never on Ethernet/PoE infra) -> ADR + label, no
  protection network.
- C J1 RJHSE-5384 footprint possible 1<->8 mirror (KiCad stock LED row reversed vs the
  Amphenol drawing) -> needs authoritative footprint resolution / physical continuity check.
- D D3 DNP: in BOM (C559105) not CPL, no machine-DNP marker -> JLC assembly defect;
  fix = populate D3 (parity-clean) or converter enhancement.
Plus P1 (GND-tail THERMAL not SOLID, NOT-ETHERNET silk not adjacent to J1, RJ45 mouth
1.05mm overhang, MK1 LCSC = MPN string) and P2 (IR-drop FIXED, jlc_twin pad_alias bug
spun off). Reproducibility: corrected r3 promoted (real audio route, DRC 0/0/0 from source;
supersedes 463fd12's stale zero-audio r3). NOT sealed.

Co-Authored-By: Claude Opus 4.8 <noreply@anthropic.com>
Routing:
- net AUDIO_P: track 0.00 -> 95.7 mm, vias 0 -> 3
- net AUDIO_N: track 0.00 -> 46.1 mm, vias 0 -> 5
- net OLB: track 8.79 -> 9.46 mm, vias 0 -> 2
- removed copper zone on B.Cu, net GND
- removed copper zone on F.Cu, net GND
