File: projects/usb-hub-3s-v3/03_src/route/final_chain.kicad_pcb (KiCad board)
At the start: 4 copper layers, 130 x 92 mm, 104 parts, among them J1 C98732, J2 C503996, J3 C503996, J4 C503996, J5 C5337088, Q1 C2760089, Q2 C404363, Q3 C404363, Q4 C404363, Q5 C404363, U10 C7519, U11 C13755, U12 C7519, U2 C13755, U3 C130056, U4 C130056, U5 C130056, U6 C473910, U7 C473910, U8 C7519, U9 C7519

Commit message: usb-hub-3s-v3 v1.1: place+route — DRC 0/0/0, protected-VBUS cell + EP vias + VBAT_F pour
DRC --severity-all --refill-zones --schematic-parity = 0/0/0. audit_board PASS,
R-THERM PASS. 119 footprints (115 parts + 4 MH). eFuse cell near J5, linear
5VC->Q6->EFINC->U13->VBUSC->J5; 5VC/EFINC/VBUSC pour split; buck-C FB Kelvin sense
on VBUSC (sense-at-connector); ENKILL to both bucks EN; snubbers (DNP). Thermal:
EP via arrays U2=7/U11=7/U13=8; VBAT_F B.Cu pour + 7 stitch vias. Delta vs v1.0:
+15 parts, SE 5VC re-topologized; buck cells/USB-A/input protection unchanged.
Adds 03_src/post_stitch_fixes.py (EP arrays/VBAT_F/floors) + vendored SW1 footprint.
Residual (verification stage): 5 policy_audit FAILs, all source-metadata (BSS138/
SS12D07 part.yaml S-VER/P-ESC/P-LAYOUT; power_tree off_control declaration for E-OFF;
DNP-snubber R-POUR) — no board defects.

Co-Authored-By: Claude Opus 4.8 <noreply@anthropic.com>
Parts:
- added C51: 10nF, Capacitor_SMD:C_0603_1608Metric, F.Cu at (110.0, 97.5)
- added C52: 100nF, Capacitor_SMD:C_0603_1608Metric, F.Cu at (108.1, 86.5)
- added C53: 1nF, Capacitor_SMD:C_0805_2012Metric, F.Cu at (88.9, 47.0)
- added C54: 1nF, Capacitor_SMD:C_0805_2012Metric, F.Cu at (88.9, 85.0)
- added Q6: C404363, Package_SO:PowerPAK_SO-8_Single, F.Cu at (104.5, 90.5)
- added Q7: C78284, Package_TO_SOT_SMD:SOT-23, F.Cu at (105.5, 98.5)
- added R30: 3.09kΩ, Resistor_SMD:R_0603_1608Metric, F.Cu at (116.5, 97.5)
- added R31: 47.5kΩ, Resistor_SMD:R_0603_1608Metric, F.Cu at (103.0, 95.6)
- added R32: 12.1kΩ, Resistor_SMD:R_0603_1608Metric, F.Cu at (106.1, 101.4)
- added R33: 100kΩ, Resistor_SMD:R_0603_1608Metric, F.Cu at (101.6, 99.2)
- added R34: 2.2Ω, Resistor_SMD:R_1206_3216Metric, F.Cu at (86.0, 44.5)
- added R35: 2.2Ω, Resistor_SMD:R_1206_3216Metric, F.Cu at (86.0, 82.5)
- added R36: 150kΩ, Resistor_SMD:R_0603_1608Metric, F.Cu at (102.8, 101.7)
- added SW1: C2939728, Button_Switch_THT:SW_Slide_1P2T_CK-12D07, F.Cu at (66.0, 58.0)
- added U13: C2866319, Package_SO:HTSSOP-20-1EP_4.4x6.5mm_P0.65mm_EP3.4x6.5mm_Mask2.75x3.43mm, F.Cu at (113.0, 92.0)
- R12, R3: value 3.74kΩ -> 3.92kΩ
- U11, U2: footprint Package_SO:HTSSOP-20-1EP_4.4x6.5mm_P0.65mm_EP3.4x6.5mm_Mask2.75x3.43mm_ThermalVias -> Package_SO:HTSSOP-20-1EP_4.4x6.5mm_P0.65mm_EP3.4x6.5mm_Mask2.75x3.43mm
- U3, U4, U5: footprint Package_SON:VSON-8-1EP_3x3mm_P0.65mm_EP1.65x2.4mm_ThermalVias -> Package_SON:VSON-8-1EP_3x3mm_P0.65mm_EP1.65x2.4mm
- moved C25 9.53 mm to (59.9, 69.1)
- moved C31 3.61 mm to (94.0, 81.5)
- moved C16 3.61 mm to (94.0, 43.5)
- moved C17 2.70 mm to (99.1, 42.6)
- moved C32 2.70 mm to (99.1, 80.6)
Connections:
- C49 pad 1: 5VC -> VBUSC
- C50 pad 1: 5VC -> VBUSC
- J5 pad A4: 5VC -> VBUSC
- J5 pad A9: 5VC -> VBUSC
- J5 pad B4: 5VC -> VBUSC
- J5 pad B9: 5VC -> VBUSC
- R12 pad 1: 5VC -> VBUSC
- R17 pad 2: EN_C -> ENKILL
- R28 pad 2: 5VC -> VBUSC
- R29 pad 2: 5VC -> VBUSC
- R8 pad 2: EN_A -> ENKILL
- U11 pad 4: EN_C -> ENKILL
- U12 pad 5: 5VC -> VBUSC
- U2 pad 4: EN_A -> ENKILL
Routing:
- net ENKILL: track 0.00 -> 67.5 mm
- net SHDNC: track 0.00 -> 27.3 mm
- net OVPC: track 0.00 -> 18.4 mm, vias 0 -> 2
- net DRVC: track 0.00 -> 16.3 mm
- net BGATEC: track 0.00 -> 15.4 mm
- net COMP_A: track 18.8 -> 11.5 mm, vias 2 -> 4
- net VCC_A: track 13.1 -> 18.3 mm
- net VCC_C: track 18.3 -> 13.1 mm
- net EN_C: track 4.85 -> 0.00 mm
- net EN_A: track 4.85 -> 0.00 mm
- net HO_A: track 20.8 -> 24.2 mm, vias 2 -> 0
- net HO_C: track 24.2 -> 20.9 mm, vias 0 -> 2
- net DVDTC: track 0.00 -> 3.04 mm
- net ILIMC: track 0.00 -> 2.75 mm
- net BOOT_A: track 14.5 -> 12.1 mm
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- added copper zone on B.Cu, net EFINC
- added copper zone on F.Cu, net EFINC
- added copper zone on B.Cu, net VBUSC
- added copper zone on F.Cu, net VBUSC
Other:
- board text added: "C51"
- board text added: "C52"
- board text added: "C53"
- board text added: "C54"
- board text added: "POWER-DIST BOARD - NOT A USB HUB"
- board text added: "PROTECTED 3S + BAL-CHG ONLY"
- board text added: "Q6"
- board text added: "Q7"
- board text added: "R30"
- board text added: "R31"
- board text added: "R32"
- board text added: "R33"
- board text added: "R34"
- board text added: "R35"
- board text added: "R36"
- board text added: "SW1"
- board text added: "U13"
- board text added: "USB-A 5V CHG no-data"
- board text added: "USB-C 5A Pi-ONLY NOT USB-PD"
- board text removed: "PROTECTED 3S PACK"
- board text removed: "USB-A 5V 2A"
- board text removed: "USB-C 5V/5A Pi"

Commit message: usb-hub-3s-v3 v1.2 routing gate (board stage) — discrete protection, DRC 0/0/0
Board stage on the re-architected discrete USB-C port protection (schematic gate
c8bc65c). The over-built TPS26631 eFuse QFN is gone, so routing converged cleanly
(the QFN pin-escape wall that failed v1.1's 5VC taps is eliminated).

Protection chain, real in-stock parts assigned:
- F2 polyfuse: BORN SMD2920-700/16N (C6165170) — 7A hold / 16V. Chosen over the
  6A 2920L600 (C3762416, kept as documented fallback) because 6A derates to
  ~4.8A @50C, below the 5A load -> nuisance-trip risk; 7A clears it.
- D5 TVS: SMBJ6.0A LRC (C140903) — Vwm 6.0V clears the 5.43V idle standoff.
- Q6 AON6403 enable-gated P-FET (Q7 BSS138 inverter on ENKILL) OFF-state
  reverse-block; buck-C FB on local 5VC.

Gate (orchestrator-verified independently, checker != checked):
- DRC 0/0/0 (--severity-all --refill-zones --schematic-parity) on the board.
- parity 110x5 (circuit.json==kicad_sch==netlist==manifest==board).
- ERC 0 errors (converter erc refreshed for the real-F2 sch).
- DIRECT M-BOM PASS: bom_source_check 06_build/fab/bom_jlc.csv vs circuit.json =
  every LCSC == source, no merged/substituted/dropped. (policy_audit's M-BOM
  FAIL is a false-positive-by-design: it compares the LATEST SEALED release BOM
  (v1.1) against v1.2 source, flagging the expected v1.1->v1.2 part changes;
  resolves at seal. Skill-refinement candidate logged.)
- route chain promoted to 03_src/route/final_chain.kicad_pcb (rebuild_fast
  reproduces 0/0/0).

Pre-seal (folded into red-team/seal, not gate blockers): discrete-protection ADR;
refresh R-THERM waiver prose (AON6354/EFINC -> AON6403 set); harvest proven-parts
(2920 PPTC + SMB TVS); ORDER_README order-day jlc_stock recheck for F2+D5 (both
Extended-tier). STATUS beacon adopted.

Co-Authored-By: Claude Opus 4.8 <noreply@anthropic.com>
Parts:
- removed C51: 10nF, Capacitor_SMD:C_0603_1608Metric
- removed C52: 100nF, Capacitor_SMD:C_0603_1608Metric
- removed R31: 47.5kΩ, Resistor_SMD:R_0603_1608Metric
- removed R32: 12.1kΩ, Resistor_SMD:R_0603_1608Metric
- removed R33: 100kΩ, Resistor_SMD:R_0603_1608Metric
- removed R36: 150kΩ, Resistor_SMD:R_0603_1608Metric
- removed U13: C2866319, Package_SO:HTSSOP-20-1EP_4.4x6.5mm_P0.65mm_EP3.4x6.5mm_Mask2.75x3.43mm
- added D5: C140903, Diode_SMD:D_SMB, F.Cu at (119.0, 96.0)
- added F2: C6165170, Fuse:Fuse_2920_7451Metric, F.Cu at (114.0, 90.0)
- Q6: value C404363 -> C2760089
- R12: value 3.92kΩ -> 4.12kΩ
- R30: value 3.09kΩ -> 100kΩ
- moved R30 8.34 mm to (108.8, 94.3)
- moved C49 4.14 mm to (121.7, 87.1)
- moved Q7 2.92 mm to (104.0, 96.0)
- moved Q6 0.71 mm to (104.0, 90.0), turned to 180 degrees
- moved C50 0.30 mm to (125.5, 91.0)
Connections:
- Q6 pad 1: 5VC -> PMID
- Q6 pad 2: 5VC -> PMID
- Q6 pad 3: 5VC -> PMID
- Q6 pad 4: BGATEC -> QG
- Q6 pad 5: EFINC -> 5VC
- Q7 pad 1: DRVC -> ENKILL
- Q7 pad 2: 5VC -> GND
- Q7 pad 3: BGATEC -> QG
- R12 pad 1: VBUSC -> 5VC
- R30 pad 1: ILIMC -> PMID
- R30 pad 2: GND -> QG
Routing:
- net ENKILL: track 67.5 -> 136.3 mm
- net SHDNC: track 27.3 -> 0.00 mm
- net OVPC: track 18.4 -> 0.00 mm, vias 2 -> 0
- net DRVC: track 16.3 -> 0.00 mm
- net BGATEC: track 15.4 -> 0.00 mm
- net QG: track 0.00 -> 12.9 mm
- net COMP_C: track 18.8 -> 13.5 mm, vias 2 -> 0
- net VCC_A: track 18.3 -> 13.1 mm
- net HO_A: track 24.2 -> 20.8 mm, vias 0 -> 2
- net DVDTC: track 3.04 -> 0.00 mm
- net ILIMC: track 2.75 -> 0.00 mm
- net BOOT_A: track 12.1 -> 14.5 mm
- net DM_A2: track 44.2 -> 41.8 mm
- net DP_A2: track 46.6 -> 48.4 mm
- net SS_A: track 6.02 -> 7.24 mm
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- added copper zone on B.Cu, net PMID
- added copper zone on F.Cu, net PMID
- added copper zone on B.Cu, net VBAT_F
- removed copper zone on B.Cu, net EFINC
- removed copper zone on F.Cu, net EFINC
Other:
- board text added: "D5"
- board text added: "F2"
- board text removed: "C51"
- board text removed: "C52"
- board text removed: "R31"
- board text removed: "R32"
- board text removed: "R33"
- board text removed: "R36"
- board text removed: "U13"
