File: projects/usb-hub-3s-v3/04_kicad/usb_hub_3s_v2.kicad_sch (KiCad schematic)
At the start: 115 parts, among them J1 C98732, J2 C503996, J3 C503996, J4 C503996, J5 C5337088, Q1 C2760089, Q2 C404363, Q3 C404363, Q4 C404363, Q5 C404363, Q6 C404363, Q7 C78284, SW1 C2939728, U10 C7519, U11 C13755, U12 C7519, U13 C2866319, U2 C13755, U3 C130056, U4 C130056, U5 C130056, U6 C473910, U7 C473910, U8 C7519, U9 C7519

Commit message: usb-hub-3s-v3 v1.2 routing gate (board stage) — discrete protection, DRC 0/0/0
Board stage on the re-architected discrete USB-C port protection (schematic gate
c8bc65c). The over-built TPS26631 eFuse QFN is gone, so routing converged cleanly
(the QFN pin-escape wall that failed v1.1's 5VC taps is eliminated).

Protection chain, real in-stock parts assigned:
- F2 polyfuse: BORN SMD2920-700/16N (C6165170) — 7A hold / 16V. Chosen over the
  6A 2920L600 (C3762416, kept as documented fallback) because 6A derates to
  ~4.8A @50C, below the 5A load -> nuisance-trip risk; 7A clears it.
- D5 TVS: SMBJ6.0A LRC (C140903) — Vwm 6.0V clears the 5.43V idle standoff.
- Q6 AON6403 enable-gated P-FET (Q7 BSS138 inverter on ENKILL) OFF-state
  reverse-block; buck-C FB on local 5VC.

Gate (orchestrator-verified independently, checker != checked):
- DRC 0/0/0 (--severity-all --refill-zones --schematic-parity) on the board.
- parity 110x5 (circuit.json==kicad_sch==netlist==manifest==board).
- ERC 0 errors (converter erc refreshed for the real-F2 sch).
- DIRECT M-BOM PASS: bom_source_check 06_build/fab/bom_jlc.csv vs circuit.json =
  every LCSC == source, no merged/substituted/dropped. (policy_audit's M-BOM
  FAIL is a false-positive-by-design: it compares the LATEST SEALED release BOM
  (v1.1) against v1.2 source, flagging the expected v1.1->v1.2 part changes;
  resolves at seal. Skill-refinement candidate logged.)
- route chain promoted to 03_src/route/final_chain.kicad_pcb (rebuild_fast
  reproduces 0/0/0).

Pre-seal (folded into red-team/seal, not gate blockers): discrete-protection ADR;
refresh R-THERM waiver prose (AON6354/EFINC -> AON6403 set); harvest proven-parts
(2920 PPTC + SMB TVS); ORDER_README order-day jlc_stock recheck for F2+D5 (both
Extended-tier). STATUS beacon adopted.

Co-Authored-By: Claude Opus 4.8 <noreply@anthropic.com>
Parts:
- removed C51: 10nF, Capacitor_SMD:C_0603_1608Metric, symbol elt:SYM_C51
- removed C52: 100nF, Capacitor_SMD:C_0603_1608Metric, symbol elt:SYM_C52
- removed R31: 47.5kΩ, Resistor_SMD:R_0603_1608Metric, symbol elt:SYM_R31
- removed R32: 12.1kΩ, Resistor_SMD:R_0603_1608Metric, symbol elt:SYM_R32
- removed R33: 100kΩ, Resistor_SMD:R_0603_1608Metric, symbol elt:SYM_R33
- removed R36: 150kΩ, Resistor_SMD:R_0603_1608Metric, symbol elt:SYM_R36
- removed U13: C2866319, Package_SO:HTSSOP-20-1EP_4.4x6.5mm_P0.65mm_EP3.4x6.5mm_Mask2.75x3.43mm, symbol elt:SYM_U13
- added D5: C140903, Diode_SMD:D_SMB, symbol elt:SYM_D5
- added F2: C6165170, Fuse:Fuse_2920_7451Metric, symbol elt:SYM_F2
- Q6: value C404363 -> C2760089
- R12: value 3.92kΩ -> 4.12kΩ
- R30: value 3.09kΩ -> 100kΩ
Connections:
- net DRVC is gone; now on net ENKILL: Q7.1 (G)
- net EFINC is gone; now on net 5VC: Q6.5 (D)
- net 5VC: now also R12.1 (pin1); no longer Q6.1 (S1), Q6.2 (S2), Q6.3 (S3), Q7.2 (S)
- net GND: now also Q7.2 (S), D5.2 (A); no longer R30.2 (pin2)
- net VBUSC: now also D5.1 (K), F2.2; no longer R12.1 (pin1)
- net BGATEC renamed QG
- net QG: now also R30.2 (pin2)
- net ILIMC renamed PMID
- net PMID: now also Q6.1 (S1), Q6.2 (S2), Q6.3 (S3), F2.1
- no-connect marks 11 -> 8
