File: projects/usb-hub-3s-v3/03_tscircuit/kicad/usb_hub_3s_v2.kicad_sch (KiCad schematic)
At the start: 100 parts, among them J1 C98732, J2 C503996, J3 C503996, J4 C503996, J5 C5337088, Q1 C2760089, Q2 C404363, Q3 C404363, Q4 C404363, Q5 C404363, U10 C7519, U11 C13755, U12 C7519, U2 C13755, U3 C130056, U4 C130056, U5 C130056, U6 C473910, U7 C473910, U8 C7519, U9 C7519

Commit message: usb-hub-3s-v3 v1.1: schematic revision — protected VBUS + 5.1V-at-connector + off-switch
v1.1 source revision (v1.0 sealed/immutable, opened read-only). ERC 0 errors;
refdes parity 115==115 (manifest/circuit/sch/netlist; +15 parts, 0 dropped;
board-lag is the immutable v1.0 board, reconciled at the board revision); E-INV 16/16.
- Protected VBUS: 5VC buck -> Q6 AON6354 (blocking) -> Q7 BSS138 (fast pulldown,
  DS-mandated 2nd FET) -> TPS26631 eFuse -> J5. ILIM 5.83A, soft-start 1.1ms,
  MODE auto-retry, OVP 5.91V cutoff, SHDN divider ~3.1V.
- FB = sense-at-connector (review preference): Buck-C senses VBUSC post-eFuse ->
  holds connector 5.151V load-independent (>=5.0V@5A, <5.25V no-load); eFuse pole
  ~234kHz >> ~20kHz crossover (comp undisturbed).
- Master-off SW1 grounds both LM5116 EN (ENKILL); caps 50V in/10V out; RC snubbers
  (DNP) on SW_A/SW_C; docs relabeled (proprietary Pi-dedicated 5A, not hub, 3S-only).
- NEW 02_parts/BSS138 (Q7, on-BOM C78284).

Co-Authored-By: Claude Opus 4.8 <noreply@anthropic.com>
Parts:
- added C51: 10nF, Capacitor_SMD:C_0603_1608Metric, symbol elt:SYM_C51
- added C52: 100nF, Capacitor_SMD:C_0603_1608Metric, symbol elt:SYM_C52
- added C53: 1nF, Capacitor_SMD:C_0805_2012Metric, symbol elt:SYM_C53
- added C54: 1nF, Capacitor_SMD:C_0805_2012Metric, symbol elt:SYM_C54
- added Q6: C404363, Package_SO:PowerPAK_SO-8_Single, symbol elt:SYM_Q6
- added Q7: C78284, Package_TO_SOT_SMD:SOT-23, symbol elt:SYM_Q7
- added R30: 3.09kΩ, Resistor_SMD:R_0603_1608Metric, symbol elt:SYM_R30
- added R31: 47.5kΩ, Resistor_SMD:R_0603_1608Metric, symbol elt:SYM_R31
- added R32: 12.1kΩ, Resistor_SMD:R_0603_1608Metric, symbol elt:SYM_R32
- added R33: 100kΩ, Resistor_SMD:R_0603_1608Metric, symbol elt:SYM_R33
- added R34: 2.2Ω, Resistor_SMD:R_1206_3216Metric, symbol elt:SYM_R34
- added R35: 2.2Ω, Resistor_SMD:R_1206_3216Metric, symbol elt:SYM_R35
- added R36: 150kΩ, Resistor_SMD:R_0603_1608Metric, symbol elt:SYM_R36
- added SW1: C2939728, Button_Switch_THT:SW_Slide_1P2T_CK-12D07, symbol elt:SYM_SW1
- added U13: C2866319, Package_SO:HTSSOP-20-1EP_4.4x6.5mm_P0.65mm_EP3.4x6.5mm_Mask2.75x3.43mm, symbol elt:SYM_U13
- R12, R3: value 3.74kΩ -> 3.92kΩ
Connections:
- net EN_C is gone; now on net ENKILL: R17.2 (pin2), U11.4 (EN)
- net 5VC: now also Q6.1 (S1), Q6.2 (S2), Q6.3 (S3), Q7.2 (S), R31.1 (pin1), R33.1 (pin1), U13.6 (IN_SYS); no longer C49.1 (pin1), C50.1 (pin1), J5.A4 (VBUSA4), J5.A9 (VBUSA9), J5.B4 (VBUSB4), J5.B9 (VBUSB9), R12.1 (pin1), R28.2 (pin2), R29.2 (pin2), U12.5 (VBUS)
- net GND: now also C51.2 (pin2), C52.2 (pin2), C53.2 (pin2), C54.2 (pin2), R30.2 (pin2), R32.2 (pin2), R36.2 (pin2), SW1.1 (T1), U13.12 (MODE), U13.16 (PGTH), U13.21 (EP), U13.7 (UVLO), U13.9 (GND)
- net SW_A: now also R34.1 (pin1)
- net SW_C: now also R35.1 (pin1)
- net EN_A renamed ENKILL
- net ENKILL: now also SW1.2 (COM)
- new net BGATEC: Q6.4 (G), Q7.3 (D), U13.4 (B_GATE)
- new net DRVC: Q7.1 (G), U13.5 (DRV)
- new net DVDTC: C51.1 (pin1), U13.10 (dVdT)
- new net EFINC: C52.1 (pin1), Q6.5 (D), U13.1 (IN), U13.2 (IN), U13.3 (IN)
- new net ILIMC: R30.1 (pin1), U13.11 (ILIM)
- new net OVPC: R31.2 (pin2), R32.1 (pin1), U13.8 (OVP)
- new net SHDNC: R33.2 (pin2), R36.1 (pin1), U13.13 (SHDN)
- new net SNUB_A: C53.1 (pin1), R34.2 (pin2)
- new net SNUB_C: C54.1 (pin1), R35.2 (pin2)
- new net VBUSC: C49.1 (pin1), C50.1 (pin1), J5.A4 (VBUSA4), J5.A9 (VBUSA9), J5.B4 (VBUSB4), J5.B9 (VBUSB9), R12.1 (pin1), R28.2 (pin2), R29.2 (pin2), U12.5 (VBUS), U13.18 (OUT), U13.19 (OUT), U13.20 (OUT)
- no-connect marks 7 -> 11

Commit message: usb-hub-3s-v3 v1.2 schematic: fix both v1.1 order-blockers (post-eFuse FB + SHDN OV)
v1.1 was DO-NOT-ORDER (2nd external review). v1.2 fixes both verified blockers:
1. Post-eFuse FB runaway: buck-C FB moved off VBUSC to LOCAL 5VC (R12 3.92k->4.12k).
   5VC regulated 5.352V; connector 5.18V typ / 5.11V hot@5A; quad-worst 5.03V >= 5.0V.
   Backed by FLT->EN (U13 FLT pin15 -> buck-C EN_C, un-merged from ENKILL; master-off
   re-coupled via D6) so a C-fault shuts only buck-C.
2. SHDN 7.56V > 5.5V abs-max: re-valued divider (R33 40.2k/R36 49.9k -> 2.96V enable)
   + Zener clamp D5 (BZT52C3V9). SHDN under 12.6V fault ~3.7V < 5.5V (margin >=1.7V).
Plus D7 (BZT52C6V2) 5VC ceiling clamp; output caps kept 10V (1.87x margin, documented).

Deviation from task: 'NFET pulldown driven by ENKILL' is wrong-polarity (ENKILL is
active-high-when-on) -> implemented the task's 'clamp SHDN' alternative (divider + hard
Zener, master-off via 5VC-collapse). Polarity proof in journal.

Gate: tsci 118 components / 382 pins / 0 dropped; GRID converter ERC 0; count_parity
118==118==118==118; E-INV 29/29; E-TOPO/E-MARGIN/E-OFF PASS; contracts_audit 0.
New parts: RT0603BRD074K12L, BZT52C3V9, BZT52C6V2 (D6 reuses 1N4148WS).

v1.2 still needs: placement+routing (new board, v1.1 04_kicad immutable) -> DRC 0/0/0
-> FRESH independent red-team (not fix-confirmation) -> seal.

Co-Authored-By: Claude Opus 4.8 <noreply@anthropic.com>
Parts:
- added D5: simple_chip, symbol elt:SYM_D5
- added D6: C2128, Diode_SMD:D_SOD-323, symbol elt:SYM_D6
- added D7: simple_chip, symbol elt:SYM_D7
- R12: value 3.92kΩ -> 4.12kΩ
- R33: value 100kΩ -> 40.2kΩ
- R36: value 150kΩ -> 49.9kΩ
Connections:
- net 5VC: now also R12.1 (pin1), D7.1 (K)
- net ENKILL: now also D6.1 (K); no longer R17.2 (pin2), U11.4 (EN)
- net GND: now also D5.2 (A), D7.2 (A)
- net SHDNC: now also D5.1 (K)
- net VBUSC: no longer R12.1 (pin1)
- net EN_C: now reaches U13.15 (FLT)
- net EN_C: now also R17.2 (pin2), U11.4 (EN), D6.2 (A)
- no-connect marks 11 -> 10

Commit message: usb-hub-3s-v3 v1.2 schematic gate (discrete protection); board stage pending
Right-size the USB-C port protection per user decision (BRIEF A2/D2): drop the
over-built TPS26631 eFuse cell (root cause of the QFN pin-escape routing wall +
v1.1 electrical blockers) for a discrete scheme that routes trivially.

New protection chain (verified from the netlist):
  5VC -> Q6 (AON6403 P-FET, D=5VC/S=PMID) -> PMID -> F2 (PPTC polyfuse) -> VBUSC -> J5
  - Q6 gate QG driven by Q7 (BSS138 inverter on ENKILL) + R30 100k pull-up to PMID:
    ON forward when hub on, OFF blocks VBUS->pack back-feed (enable-gated P-FET,
    NOT an ideal-diode controller).
  - D5 SMBJ6.0A TVS on VBUSC->GND (over-voltage).
  - buck-C FB R12.1 = 5VC (local-sense v1.1 fix kept).

Refdes 118 -> 110: removed U13 (TPS26631) + R31/R32/R33/R36/C51/C52/D6/D7;
added F2; re-roled Q6->AON6403, R30->100k gate pull-up, D5->SMBJ6.0A TVS,
Q7->ENKILL inverter. Removed part folders TPS26631PWPR, BZT52C3V9, BZT52C6V2.

Schematic gate (orchestrator-verified independently): ERC 0 errors (fresh
kicad-cli sch erc on the regenerated converter sch; erc_converter.rpt refreshed
in-place, no stale eFuse refs), parity 110==110==110==110 (circuit.json ==
kicad_sch == netlist == manifest), E-INV 24/24, contracts 0.

Board stage pending: floorplan.yaml / route.yaml / rules/nets.yaml / 04_kicad
still hold eFuse-era seeds+keepouts+asserts and the stale DRC board; they get
ripped out and re-derived from the 110-comp schematic in the board stage.
Stock caveat: F2 polyfuse (MF-MSMF600 candidate has Vmax=6V, INSUFFICIENT vs the
12.6V buck-fail-high case) + D5 TVS need real in-stock LCSC assignment before seal.

Co-Authored-By: Claude Opus 4.8 <noreply@anthropic.com>
Parts:
- removed C51: 10nF, Capacitor_SMD:C_0603_1608Metric, symbol elt:SYM_C51
- removed C52: 100nF, Capacitor_SMD:C_0603_1608Metric, symbol elt:SYM_C52
- removed D6: C2128, Diode_SMD:D_SOD-323, symbol elt:SYM_D6
- removed D7: simple_chip, symbol elt:SYM_D7
- removed R31: 47.5kΩ, Resistor_SMD:R_0603_1608Metric, symbol elt:SYM_R31
- removed R32: 12.1kΩ, Resistor_SMD:R_0603_1608Metric, symbol elt:SYM_R32
- removed R33: 40.2kΩ, Resistor_SMD:R_0603_1608Metric, symbol elt:SYM_R33
- removed R36: 49.9kΩ, Resistor_SMD:R_0603_1608Metric, symbol elt:SYM_R36
- removed U13: C2866319, Package_SO:HTSSOP-20-1EP_4.4x6.5mm_P0.65mm_EP3.4x6.5mm_Mask2.75x3.43mm, symbol elt:SYM_U13
- added F2: C2828687, Fuse:Fuse_1812_4532Metric, symbol elt:SYM_F2
- D5: value simple_chip -> C921382; footprint (none) -> Diode_SMD:D_SMB
- Q6: value C404363 -> C2760089
- R30: value 3.09kΩ -> 100kΩ
Connections:
- net DRVC is gone; now on net ENKILL: Q7.1 (G)
- net EFINC is gone; now on net 5VC: Q6.5 (D)
- net EN_C is gone; now on net ENKILL: R17.2 (pin2), U11.4 (EN)
- net SHDNC is gone; now on net VBUSC: D5.1 (K)
- net 5VC: no longer Q6.1 (S1), Q6.2 (S2), Q6.3 (S3), Q7.2 (S)
- net GND: now also Q7.2 (S); no longer R30.2 (pin2)
- net VBUSC: now also F2.2
- net BGATEC renamed QG
- net QG: now also R30.2 (pin2)
- net ILIMC renamed PMID
- net PMID: now also Q6.1 (S1), Q6.2 (S2), Q6.3 (S3), F2.1
- no-connect marks 10 -> 8

Commit message: usb-hub-3s-v3 v1.2 routing gate (board stage) — discrete protection, DRC 0/0/0
Board stage on the re-architected discrete USB-C port protection (schematic gate
c8bc65c). The over-built TPS26631 eFuse QFN is gone, so routing converged cleanly
(the QFN pin-escape wall that failed v1.1's 5VC taps is eliminated).

Protection chain, real in-stock parts assigned:
- F2 polyfuse: BORN SMD2920-700/16N (C6165170) — 7A hold / 16V. Chosen over the
  6A 2920L600 (C3762416, kept as documented fallback) because 6A derates to
  ~4.8A @50C, below the 5A load -> nuisance-trip risk; 7A clears it.
- D5 TVS: SMBJ6.0A LRC (C140903) — Vwm 6.0V clears the 5.43V idle standoff.
- Q6 AON6403 enable-gated P-FET (Q7 BSS138 inverter on ENKILL) OFF-state
  reverse-block; buck-C FB on local 5VC.

Gate (orchestrator-verified independently, checker != checked):
- DRC 0/0/0 (--severity-all --refill-zones --schematic-parity) on the board.
- parity 110x5 (circuit.json==kicad_sch==netlist==manifest==board).
- ERC 0 errors (converter erc refreshed for the real-F2 sch).
- DIRECT M-BOM PASS: bom_source_check 06_build/fab/bom_jlc.csv vs circuit.json =
  every LCSC == source, no merged/substituted/dropped. (policy_audit's M-BOM
  FAIL is a false-positive-by-design: it compares the LATEST SEALED release BOM
  (v1.1) against v1.2 source, flagging the expected v1.1->v1.2 part changes;
  resolves at seal. Skill-refinement candidate logged.)
- route chain promoted to 03_src/route/final_chain.kicad_pcb (rebuild_fast
  reproduces 0/0/0).

Pre-seal (folded into red-team/seal, not gate blockers): discrete-protection ADR;
refresh R-THERM waiver prose (AON6354/EFINC -> AON6403 set); harvest proven-parts
(2920 PPTC + SMB TVS); ORDER_README order-day jlc_stock recheck for F2+D5 (both
Extended-tier). STATUS beacon adopted.

Co-Authored-By: Claude Opus 4.8 <noreply@anthropic.com>
Parts:
- D5: value C921382 -> C140903
- F2: value C2828687 -> C6165170; footprint Fuse:Fuse_1812_4532Metric -> Fuse:Fuse_2920_7451Metric

Commit message: usb-hub-3s-v3 v1.3 gate (i): catalog-verified R12 + D5, setpoint re-derived, OV honesty
Fix-pass checkpoint on the SUPERSEDED v1.2 (39c5767). Schematic/BOM-side only;
board+artifact regen is gate (ii).

R12 (the confirmed order blocker): C2984354 (AR03BTCX4121, Viking) CATALOG-
VERIFIED 4.12k +/-0.1% +/-25ppm, 15,353 stock — BAKED in the tsx as an explicit
MPN so tscircuit can never value-resolve back to the 3.74k C2933210 (the bug;
now 0 occurrences). C861436 verified drop-in alternate. Part folder renamed
RT0603BRD074K12L -> AR03BTCX4121. Orchestrator-verified: circuit.json R12 =
{resistance 4120, jlcpcb C2984354}; MPN encoding independently confirms 4121 ->
4.12k (the semantic check the old M-BOM lacked).

Setpoint RE-DERIVED against the ACTUAL Q6+F2 path (removed-eFuse IR model
dropped from power_tree.yaml): 5.352V nom, ir_budget 88mOhm (Q6 4.3 + F2 R1max
18 catalog-verified + board/conn/cable), E-MARGIN PASS 112mV slack. The 3.74k
case now FAILS E-MARGIN (265 < 528mV) — the gate itself catches the incident class.

D5 was a REAL second defect (external reviewer right): C140903 is catalog-listed
BIDIRECTIONAL (no cathode -> the D5.1=VBUSC unidirectional assertion was
unverifiable). Replaced with C113976 — SMBJ6.0A UNIDIRECTIONAL (MPN A-suffix,
not CA), same SMB footprint, Vwm 6.0/Vbr 7.37/Vclamp 10.3, 74,758 stock — baked
in tsx + part.yaml + twin_adjudications + ADR-0002.

OV honesty: BRIEF A3/D3 records the user decision with the escalation boundary
verbatim ("add active OVP if the system becomes unattended, hard-access, carries
valuable storage, or powers expensive SDR"); ADR-0002/ARCHITECTURE/E-INV state
D5/F2 = SECONDARY/best-effort; no doc claims fail-high protection (swept).
Bonus: ARCHITECTURE.md still described the removed eFuse as current protection —
updated to the discrete chain.

Checkpoint gates (orchestrator-verified): tsci build OK, converter 110/110 FPID,
fresh ERC 0.

Co-Authored-By: Claude Opus 4.8 <noreply@anthropic.com>
Parts:
- D5: value C140903 -> C113976
Connections:
- net VCC_A is gone; now on net BOOT_A: C8.1, D3.2 (A), U2.16 (VCC)
- net VCC_C is gone; now on net BOOT_C: C23.1, D4.2 (A), U11.16 (VCC)

Commit message: usb-hub-3s-v3 v1.3 gate (ii): board+artifact regen, SW1+F1 off-CPL (fix pass)
Independently verified: DRC 0/0/0 (severity-all+refill-zones+schematic-
parity, re-run directly on 04_kicad source), sha256 self-check 36/36,
git-check-ignore sweep clean on staged release dir.

Board regen from committed v1.3 gate-(i) source (R12=C2984354 4.12k,
D5=C113976 unidirectional): grid-mode converter -> netlist -> E-INV 24/24
-> rebuild_fast (promoted chain) -> DRC 0/0/0. SW1 (pitch-unconfirmed,
hand-solder) and F1 holder (hand-solder since v1.1, previously
erroneously machine-placed) both marked EXCLUDE_FROM_POS_FILES via new
floorplan patterns block. BOM 44 lines / CPL 108 placements. Full fab/
PDF/STEP/audit/twin regen staged at 07_releases/v1.3-2026-07-23 (37
files): policy_audit FAIL=0 (28 PASS/2 WAIVED/6 HUMAN/2 N-A), jlc_twin
87 OK/233 exit 0 zero unadjudicated, bom_source_check PASS (BOM delta
vs v1.2 = exactly R12+D5), release_freshness_check PASS.

MANIFEST git_sha still reads ecd82c0 (gate-i); next commit re-stamps
it to this commit + re-clears M-REL via policy_audit --skip-drc.

Co-Authored-By: Claude Opus 4.8 <noreply@anthropic.com>
Connections:
- net BOOT_A: no longer C8.1, D3.2 (A), U2.16 (VCC)
- net BOOT_C: no longer C23.1, D4.2 (A), U11.16 (VCC)
- new net VCC_A: C8.1 (pin1), D3.2 (A), U2.16 (VCC)
- new net VCC_C: C23.1 (pin1), D4.2 (A), U11.16 (VCC)
