File: projects/usb-hub-3s-v3/03_tscircuit/kicad/usb_hub_3s_v2.kicad_sch (KiCad schematic)
At the start: 110 parts, among them J1 C98732, J2 C503996, J3 C503996, J4 C503996, J5 C5337088, Q1 C2760089, Q2 C404363, Q3 C404363, Q4 C404363, Q5 C404363, Q6 C2760089, Q7 C78284, SW1 C2939728, U10 C7519, U11 C13755, U12 C7519, U2 C13755, U3 C130056, U4 C130056, U5 C130056, U6 C473910, U7 C473910, U8 C7519, U9 C7519

Commit message: usb-hub-3s-v3 v1.6: DRC 0/0/0 — the H3 screw-short is gone, and 11 CPL rows were off JLC's datum
v1.5 is DO-NOT-ORDER, and not for a reason any render could show. A new A-POS
gate measured every CPL row against JLC's convention — JLC positions a part
from the bounding box of its PAD CENTRES — and found the exporter had been
emitting fp.GetPosition(), the footprint ANCHOR. 11 of 108 rows were off-datum:
J1 4.6861mm, J2/J3/J4 3.7346mm, J5 1.4975mm, Q4/Q5/Q6 0.0625mm. Every external
connector, worst by nearly 5mm.

COPPER, all measured on FILLED zones before and after.

H3 was a short of the 6A rail to GND through a screw. MEASURED on sealed v1.5:
H3 (106,24) is a 1.600mm-radius NPTH whose F.Cu carries GND at 1.850mm AND 5VA
at 1.850mm, and whose B.Cu carries 5VA at 1.850 AND GND at 1.851. 0.250mm of
bare laminate and ~20um of mask, on both faces. EVERY M3 fastener bridges it —
not just a big washer, the smallest cap head (r 2.75) already does. v1.5's only
mitigation was a sentence in ORDER_README about nylon standoffs, which survives
exactly as long as the person who read it.

So v1.6 states a RULE instead of a note: within r <= 4.00mm of any mounting
hole, all outer copper is ONE net and that net is GND. Enforced three ways —
the 5VA pour is notched (5VA now stops at 4.500mm), the router's hole keepout
goes 3.0 -> 4.2mm so a signal wave cannot re-create it on a different net, and
the check is re-measured on the final filled board rather than assumed.

Also: H4's VBUSA3 4.152 -> 5.008mm (a DIN 9021 washer reached it); the In2 VIN
plane 1.850 -> 2.077mm on all four drills (0.250mm to a 12.6V plane, against a
+-0.13mm NPTH position tolerance, buried where no inspection will ever see it).
In1 GND is deliberately left at 1.850 — a grounded fastener touching GND is the
benign case and thinning the return plane costs more than it buys.

VBUS ampacity 0.5 -> 0.8mm. "Pour-fed" was true of the connector end and false
of the feed: each of VBUSA1/2/3 ran 13.554mm of 0.500mm B.Cu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
Parts:
- added D10: C2297, LED_SMD:LED_0805_2012Metric, symbol elt:SYM_D10
- added D11: C2297, LED_SMD:LED_0805_2012Metric, symbol elt:SYM_D11
- added D12: C2297, LED_SMD:LED_0805_2012Metric, symbol elt:SYM_D12
- added D8: C2296, LED_SMD:LED_0805_2012Metric, symbol elt:SYM_D8
- added D9: C2297, LED_SMD:LED_0805_2012Metric, symbol elt:SYM_D9
- added Q8: C78284, Package_TO_SOT_SMD:SOT-23, symbol elt:SYM_Q8
- added R37: 6.98kΩ, Resistor_SMD:R_0603_1608Metric, symbol elt:SYM_R37
- added R38: 6.98kΩ, Resistor_SMD:R_0603_1608Metric, symbol elt:SYM_R38
- added R39: 6.98kΩ, Resistor_SMD:R_0603_1608Metric, symbol elt:SYM_R39
- added R40: 6.98kΩ, Resistor_SMD:R_0603_1608Metric, symbol elt:SYM_R40
- added R41: 6.98kΩ, Resistor_SMD:R_0603_1608Metric, symbol elt:SYM_R41
- Q1, Q2, Q3, Q4, Q5, Q6: footprint Package_SO:PowerPAK_SO-8_Single -> usb_hub_3s:PowerPAK_SO-8_Single_Paste65
Connections:
- net ENKILL: now also Q8.1 (G)
- net GND: now also D10.1 (K), D11.1 (K), D12.1 (K), D9.1 (K), Q8.2 (S)
- net VBUSA1: now also R38.1 (pin1)
- net VBUSA2: now also R39.1 (pin1)
- net VBUSA3: now also R40.1 (pin1)
- net VBUSC: now also R41.1 (pin1)
- net VIN: now also R37.1 (pin1)
- new net LEDPK: D8.2 (A), R37.2 (pin2)
- new net LEDPKK: D8.1 (K), Q8.3 (D)
- new net LEDVA1: D9.2 (A), R38.2 (pin2)
- new net LEDVA2: D10.2 (A), R39.2 (pin2)
- new net LEDVA3: D11.2 (A), R40.2 (pin2)
- new net LEDVC: D12.2 (A), R41.2 (pin2)
