File: projects/pluto-cal-switch/04_kicad/pluto_cal_switch.kicad_sch (KiCad schematic)
At the start: 73 parts, among them Y1 C20625731

Commit message: the header divider was INVERTED, and the published table is what proved it was a transposition and not an estimate
R_HDR_S 2.2k / R_HDR_G 3.3k gives 3.3/(2.2+3.3) = 0.600*Vin. ADR-0008,
ARCHITECTURE, DETAIL_DESIGN and the tsx comment all published 0.400 and
tabulated 0.72 / 1.32 / 2.00 V. Those are not approximations of 0.600 —
they are EXACTLY the voltages the two values produce when swapped, which
is what makes this a transposition with a known correct answer rather
than a disagreement to be split.

Verified as-built before touching anything, in the netlist and not in the
prose: tsc_netlist.txt HDR_CTRL_IN -[R_HDR_S 2.2k]- HDR_CTRL_ADC
-[R_HDR_G 3.3k]- GND.

SWAPPED rather than re-documented, on three grounds:
  * the ratio the ADR argues for throughout is /2.5;
  * it TIGHTENS the fault bound the ADR already claims — a firmware bug
    driving 3.3 V into a clamped 1.8 V Zynq pin sources (3.3-2.3)/3.3k =
    0.303 mA, not the 0.45 mA the ADR credited to 2.2k;
  * the defect is the CEILING, not the detect threshold. At 0.600 the
    0.36 V threshold clears with BETTER margin (1.080 V at a 1.8 V
    header) — which is why no functional test finds it — but a 5.0 V
    header reads 3.000 V against a 3.3 V ADC full scale: 0.30 V of
    headroom, ~0.23 V against a -2 % ADC_AVDD of 3.234 V. At the
    USB-legal 5.5 V it reads 3.300 V, AT or ABOVE AVDD, forward-biasing
    the input ESD diode. At 0.400 the same 5.5 V reads 2.200 V.

BOM-NEUTRAL: C25879 (2.2k) and C137992 (3.3k) are each used exactly once
and only here, so the swap moves which refdes takes which reel and
changes no line-item quantity. bom_source_check PASS confirms the
LCSC-to-value join after the swap.

WHY NOTHING CAUGHT IT, AND WHAT NOW DOES. The only assert on the divider
was `part_value R_HDR_S min: 1k`, which 2.2k satisfies. Existence was
pinned (net_has_part: 2 resistors on HDR_CTRL_ADC) and one value was
floored, and neither pins a RATIO. Now pinned by two asserts that pin two
different things, bec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
Parts:
- R_HDR_G: value 3.3kΩ -> 2.2kΩ
- R_HDR_S: value 2.2kΩ -> 3.3kΩ
