File: projects/programmable-usb2-hub/03_src/route/final_chain.kicad_pcb (KiCad board)
At the start: 4 copper layers, 130 x 90 mm, 206 parts, among them J1 C8404, J2 C86462, J3 USB1130-15-A, J4 USB1130-15-A, J5 USB1130-15-A, J6 USB1130-15-A, J7 C19191796, Q1 C454269, Q2 C454269, Q3 C404363, Q4 C404363, Q5 C404363, Q6 C404363, U1 C3215601, U10 C3662799, U11 C3662799, U12 C3662799, U13 C11355, U14 C11355, U15 C11355, U16 C11355, U17 C7519, U18 C7519, U19 C7519, U2 C13755, U20 C7519, U3 C13755, U4 C780769, U5 C7519, U6 C478081, U7 C2847904, U8 C6053, U9 C3662799, Y1 C1985204

Commit message: Preserve USB hub redesign and pipeline groundwork
Parts:
- L3: value C307880 -> C266428; footprint Inductor_SMD:L_TDK_VLS6045EX_VLS6045AF -> Inductor_SMD:L_Sunlord_SWPA6028S
- moved C115 29.6 mm to (103.8, 79.1)
- moved C114 29.3 mm to (81.2, 97.8)
- moved C23 27.5 mm to (75.2, 76.0), turned to 180 degrees
- moved C24 26.8 mm to (80.0, 76.0)
- moved C21 23.0 mm to (67.0, 85.2)
- moved R414 12.4 mm to (53.2, 46.8), turned to -90 degrees
- moved C432 10.6 mm to (110.8, 48.5), turned to -90 degrees
- moved C422 9.40 mm to (79.0, 47.2), turned to 180 degrees
- moved R444 7.68 mm to (136.3, 42.2), turned to 180 degrees
- moved R434 7.25 mm to (108.8, 42.0), turned to 90 degrees
- moved R424 6.22 mm to (81.0, 42.2), turned to 90 degrees
- moved C442 4.26 mm to (133.2, 42.2), turned to 180 degrees
- moved C441 1.77 mm to (132.5, 40.6), turned to 180 degrees
- moved C412 1.60 mm to (50.8, 48.0), turned to 180 degrees
- moved R422 1.03 mm to (85.5, 39.8), turned to 90 degrees
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Routing:
- net VIN_PROTECTED: track 248.4 -> 208.3 mm
- net 5V_B: track 156.1 -> 174.9 mm, vias 15 -> 17
- net P1_ILIM: track 26.3 -> 18.0 mm, vias 7 -> 5
- net P3_ILIM: track 24.3 -> 16.3 mm
- net P4_ITIMER: track 7.54 -> 14.8 mm
- net 5V_A: track 192.5 -> 185.9 mm, vias 19 -> 18
- net P4_ILIM: track 15.5 -> 12.2 mm, vias 4 -> 3
- net P2_ILIM: track 16.4 -> 13.9 mm
- net 3V3_LOGIC: track 409.1 -> 410.9 mm
- net GND: vias 66 -> 70
- net P2_VBUS: vias 5 -> 4
Other:
- board text added: "12-24V + -"
- board text added: "SWD"
- board text removed: "12-24V DC + -"
