File: projects/pluto-rx2-8way-v5/03_tscircuit/kicad/pluto_rx2_8way_v5.kicad_sch (KiCad schematic)
At the start: 29 parts, among them J1 C5184243, J10 C429844, J11 C2932107, J2 C429844, J3 C429844, J4 C429844, J5 C429844, J6 C429844, J7 C429844, J8 C429844, J9 C429844, U1 C5121458, U2 C5452432, U3 C2866134, U4 C1972959

Commit message: Add Pluto bench power and correct SMA renders
Parts:
- added J12: C225477, Connector_PinHeader_2.54mm:PinHeader_1x02_P2.54mm_Vertical, symbol elt:SYM_J12
Connections:
- net GND: now also J12.2 (GND)
- net VBUS_RAW: now also J12.1 (BENCH_5V)
