File: projects/usb-controlled-debug-hub-v1/03_tscircuit/kicad/usb_controlled_debug_hub.kicad_sch (KiCad schematic)
At the start: 139 parts

Commit message: Complete debug hub routing and release gates
Other:
- title: usb_controlled_debug_hub -> usb_controlled_debug_hub.fresh

Commit message: fix USB debug hub power sense and connector orientation
Parts:
- R_VBUS_TOP: value 100kΩ -> 47kΩ
Other:
- title: usb_controlled_debug_hub.fresh -> usb_controlled_debug_hub
