File: projects/usb-controlled-debug-hub-2a-v1/04_kicad/usb_controlled_debug_hub_2a.kicad_pcb (KiCad board)
At the start: 4 copper layers, 150 x 115 mm, 190 parts

Commit message: repair 2A debug hub USB routing and release gates
Routing:
- net PWR_EN4: track 68.9 -> 86.3 mm, vias 4 -> 12
- net PWR_EN2: track 77.4 -> 94.2 mm, vias 4 -> 9
- net VBUS_CTRL: track 123.5 -> 139.5 mm, vias 14 -> 17
- net 3V3_MAIN: track 397.3 -> 413.2 mm, vias 35 -> 36
- net P5V_B_PROTECTED: track 46.3 -> 57.6 mm, vias 36 -> 34
- net UP_HUB_P: track 110.6 -> 117.6 mm, vias 3 -> 5
- net UP_HUB_N: track 110.6 -> 116.5 mm, vias 4 -> 6
- net HUB_OCS2_N: track 56.0 -> 61.3 mm
- net HUB_OCS1_N: track 51.8 -> 56.4 mm, vias 6 -> 8
- net GND: track 75.2 -> 71.7 mm, vias 190 -> 189
- net HUB_OCS3_N: track 26.0 -> 28.9 mm
- net P4_HUB_P: track 98.6 -> 101.5 mm
- net PWR_EN3: track 77.8 -> 75.3 mm, vias 4 -> 11
- net DATA_OK4: track 58.7 -> 56.9 mm, vias 2 -> 6
- net I2C_SCL: track 54.8 -> 56.4 mm, vias 5 -> 6
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